File: Architecture/Main/uc.kicad_sch (KiCad schematic)
At the start: 3 parts

Commit message: Archi_1
Connections:
- net D18 is gone; now on net VIN: U1. (3.3V)
- net D19 is gone; now on net VIN: U1. (3.3V)
- net D23 is gone; now on net VIN: U1. (3.3V)
- net D5 is gone; now on net VIN: U1. (3.3V)
- new net CS: U1. (3.3V)
- new net MISO: U1. (3.3V)
- new net MOSI: U1. (3.3V)
- new net SCK: U1. (3.3V)
Other:
- moved on the sheet: U1

Commit message: Archi_2
Connections:
- net CS is gone; now on net VIN: U1. (3.3V)
- new net CS_SD: U1. (3.3V)
Other:
- moved on the sheet: R1, R2, U1

Commit message: Update Schematic
Connections:
- new net D16: U1. (3.3V)
- new net D17: U1. (3.3V)
Changed lines of the file:
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@@
 	(wire
 		(pts
+			(xy 187.96 91.44) (xy 194.31 91.44)
+		)
+		(stroke
+			(width 0)
+			(type default)
+		)
+	)
+	(wire
+		(pts
 			(xy 187.96 83.82) (xy 194.31 83.82)
 		)
@@
 	(wire
 		(pts
+			(xy 187.96 88.9) (xy 194.31 88.9)
+		)
+		(stroke
+			(width 0)
+			(type default)
+		)
+	)
+	(wire
+		(pts
 			(xy 160.02 86.36) (xy 162.56 86.36)
 		)
@@
 		)
 	)
+	(hierarchical_label "D17"
+		(shape input)
+		(at 194.31 88.9 0)
+		(effects
+			(font
+				(size 1.27 1.27)
+			)
+			(justify left)
+		)
+	)
 	(hierarchical_label "SCK"
 		(shape input)
@@
 		)
 	)
+	(hierarchical_label "D16"
+		(shape input)
+		(at 194.31 91.44 0)
+		(effects
+			(font
+				(size 1.27 1.27)
+			)
+			(justify left)
+		)
+	)

Commit message: Update
Connections:
- net CS_SD is gone; now on net VIN: U1. (3.3V)
- net D12 is gone; now on net VIN: U1. (3.3V)
- net D13 is gone; now on net VIN: U1. (3.3V)
- net D14 is gone; now on net VIN: U1. (3.3V)
- net D15 is gone; now on net VIN: U1. (3.3V)
- net D16 is gone; now on net VIN: U1. (3.3V)
- net D17 is gone; now on net VIN: U1. (3.3V)
- net D24 is gone; now on net VIN: U1. (3.3V)
- net MISO is gone; now on net VIN: U1. (3.3V)
- net MOSI is gone; now on net VIN: U1. (3.3V)
- net RX0 is gone; now on net VIN: U1. (3.3V)
- net SCK is gone; now on net VIN: U1. (3.3V)
- net TX0 is gone; now on net VIN: U1. (3.3V)
- new net D1: U1. (3.3V)
- new net D12_MISO: U1. (3.3V)
- new net D13_MOSI: U1. (3.3V)
- new net D14_CLK: U1. (3.3V)
- new net D15_CS: U1. (3.3V)
- new net D18: U1. (3.3V)
- new net D19: U1. (3.3V)
- new net D23: U1. (3.3V)
- new net D27: U1. (3.3V)
- new net D3: U1. (3.3V)
- new net D5: U1. (3.3V)
- new net RX2: U1. (3.3V)
- new net TX2: U1. (3.3V)
