File: Architecture/Main/Main.kicad_sch (KiCad schematic)
At the start: 1 part, among them U4 PCA9555D

Commit message: Archi_1
Parts:
- removed U4: PCA9555D, Package_SO:SOIC-24W_7.5x15.4mm_P1.27mm, symbol Interface_Expansion:PCA9555D
Other:
- added sheet Stockage (Stockage.kicad_sch)
- sheet Sensors ports: added D36, RX0, TX0; removed none
- sheet uc ports: added CS, MISO, MOSI, SCK; removed none

Commit message: Archi_2
Connections:
- no-connect marks 1 -> 0
Other:
- sheet Cam ports: added CS_CAM, IR, MISO, MOSI, SCK, SCL, SDA; removed D0, D1, D2, D3, D4, D5, D6, D7, HREF, I2C_SCL, I2C_SDA, PCLK, PWD, VREF, XCLK, nRST
- sheet Power ports: added +3.3V_BATT, +3.3V_POWER_UP, PWR_U/D; removed +3.3V, VIN
- sheet Sensors ports: added DATA_DHT22, MOUV; removed none
- sheet uc ports: added CS_SD; removed CS, D18, D19, D23, D5
- company: (none) -> Polytech Nantes - ETN4
- title: (none) -> Collecteur de données Animalières

Commit message: Update Schematic
Other:
- sheet Cam ports: added D0, D1, D2, D3, D4, D5, D6, D7, DCLK, HREF, LED_IR_PWR, PWDN, RST, VREF; removed CS_CAM, MISO, MOSI, SCK
- sheet uc ports: added D16, D17; removed none

Commit message: Update
Connections:
- no-connect marks 0 -> 2
Other:
- sheet Power ports: added PIR_MOUV; removed none
- sheet Sensors ports: added BRIGHTNESS_SENSOR; removed D36, MOUV
- sheet uc ports: added D1, D12_MISO, D13_MOSI, D14_CLK, D15_CS, D18, D19, D23, D27, D3, D5, RX2, TX2; removed CS_SD, D12, D13, D14, D15, D16, D17, D24, MISO, MOSI, RX0, SCK, TX0

Commit message: update
Connections:
- no-connect marks 2 -> 3
Other:
- sheet Power ports: added none; removed PIR_MOUV

Commit message: Update_07_01_2026
Connections:
- no-connect marks 3 -> 4
Other:
- sheet Cam ports: added 12V; removed LED_IR_PWR
- sheet Power ports: added 12V_POWER_UP, PIR_MOUV, WAKE_UP; removed none
- sheet Sensors ports: added +3.3V_BATTERY, PIR_MOUV; removed none

Commit message: CodeFinalProto_plus_majarchitecture
Other:
- sheet Sensors ports: added Voltage_Batt; removed none
Changed lines of the file:
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@@
+	(wire
+		(pts
+			(xy 69.85 58.42) (xy 130.81 58.42)
+		)
+		(stroke
+			(width 0)
+			(type default)
+		)
+	)
 	(wire
 		(pts
@@
 			)
 		)
+		(pin "Voltage_Batt" input
+			(at 69.85 58.42 0)
+			(effects
+				(font
+					(size 1.27 1.27)
+				)
+				(justify right)
+			)
+		)
 		(instances
 			(project "Main"
@@
 		)
 		(pin "D2" input
-			(at 177.8 52.07 0)
-			(effects
-				(font
-					(size 1.27 1.27)
-				)
-				(justify right)
-			)
-		)
+			(at 130.81 58.42 180)
+			(effects
+				(font
+					(size 1.27 1.27)
+				)
+				(justify left)
+			)
+		)

Commit message: Update_She
Connections:
- no-connect marks 4 -> 5
Other:
- sheet Cam ports: added none; removed IR
- sheet Power ports: added RECHARGE_INFO, VOLTAGE_BAT; removed WAKE_UP
- sheet Sensors ports: added Voltage_Batt_value; removed none
- sheet uc ports: added CLK, CS, MISO, MOSI; removed D12_MISO, D13_MOSI, D14_CLK, D15_CS
