File: Architecture/Main/Power.kicad_sch (KiCad schematic)
At the start: 4 parts, among them J1 Batt, J2 Panneau

Commit message: Archi_2
Parts:
- removed D2: D, symbol Device:D
- removed J2: Panneau, symbol Connector:Screw_Terminal_01x02
- added Q1: PMOS, symbol Simulation_SPICE:PMOS
- added Q2: NPN, symbol Simulation_SPICE:NPN
- added R7, R8, R9: R_US, Resistor_SMD:R_0805_2012Metric_Pad1.20x1.40mm_HandSolder, symbol Device:R_US
Connections:
- net GND: now also Q2.3 (E)
- new net: Q2.1 (C), R8.2
- new net: Q2.2 (B), R9.2
- new net: Q1.2 (G), R7.2, R8.1
- new net +3.3V_BATT: Q1.1 (D), R7.1
- new net +3.3V_POWER_UP: Q1.3 (S)
- new net PWR_U/D: R9.1
Other:
- note added: "POWER UP AND DOWN, DRIVE WITH GPIO"
- moved on the sheet: D1, J1

Commit message: Power Sector Update
Parts:
- added C1: 22u, symbol Device:C_Polarized
- added C2, C3: 220u, symbol Device:C_Polarized
- added D1, D2, D3, D4, D5: D, symbol Device:D
- added L1: 68u, symbol Device:L
- added R1: 3.01k, symbol Device:R_US
- added R2: 1.78k, symbol Device:R_US
- added U1: MIC4690, Package_SO:SOIC-8_3.9x4.9mm_P1.27mm, symbol Regulator_Switching:MIC4690
- J1: value Batt -> 12V - Secteur
- R7: value R_US -> 100k
- R8: value R_US -> 10k
- R9: value R_US -> 1k
Connections:
- net +3.3V_BATT: now also D4.1 (K), D5.1 (K)
- net +3.3V_POWER_UP: now also C3.1
- net GND: now also J1.1 (Pin_1), C1.2, C2.2, C3.2, D1.2 (A), R2.2, U1.1 (SHDN), U1.5 (GND), U1.6 (GND), U1.7 (GND), U1.8 (GND)
- net PWR_U/D: now also D2.2 (A); no longer R9.1
- net at D1.1 (K): now also C1.1, U1.2 (VIN)
- net at D1.2 (A): now also J1.2 (Pin_2)
- new net: D2.1 (K), D3.1 (K), R9.1
- new net: R1.2, R2.1, U1.4 (FB)
- new net: D1.1 (K), L1.1, U1.3 (SW)
- new net: C2.1, D4.2 (A), L1.2, R1.1
- new net PIR_MOUV: D3.2 (A)
Other:
- note added: "https://www.microchip.com/en-us/parametric-search/418?filters=JTdCJTIyYWN0aXZlU2xpZGVyRmlsdGVycyUyMiUzQSU1QiU1QiUyMlZJTiUyME1pbiUyMFYlMjAodm9sdCklMjIlMkMlNUI0LjIlMkMyLjIlNUQlNUQlNUQlMkMlMjJjYXRlZ29yeWRyb3Bkb3duJTIyJTNBJTVCJTIyUG93ZXIlMjBNYW5hZ2VtZW50JTIyJTJDJTIyREMtREMlMjBCb29zdCUyMChTdGVwLVVwKSUyMFN3aXRjaGluZyUyMENvbnZlcnRlcnMlMjIlMkMlMjJCdWNrJTIwU3dpdGNoaW5nJTIwQ29udmVydGVycyUyMCVFMiU4MCU5MyUyM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"
- note removed: "POWER UP AND DOWN, DRIVE WITH GPIO"
- moved on the sheet: D1, J1, Q1, Q2, R7, R8, R9

Commit message: Update
Parts:
- renumbered C3 to C?, C2 to C?, C1 to C?, D2 to D?, D5 to D?, D1 to D?, D3 to D?, D4 to D?, L1 to L?, R2 to R?, R1 to R?, U1 to U?
Changed lines of the file:
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@@
 		(dnp no)
 		(fields_autoplaced yes)
-		(property "Reference" "Q?"
+		(property "Reference" "Q2"
 			(at 198.12 53.3399 0)
 			(effects
@@
 		(dnp no)
 		(fields_autoplaced yes)
-		(property "Reference" "C3"
+		(property "Reference" "C?"
 			(at 220.98 44.8309 0)
 			(effects
@@
 		)
 		(instances
+			(project "Main"
+				(path "/77f264da-4c84-4b0c-9d20-4392731765e6/8078826c-4446-4e50-a209-45fcf7cbe7e4"
+					(reference "C?")
+					(unit 1)
+				)
+			)
 			(project "Power"
 				(path "/7fd1e59d-d896-4263-8d21-df7365fed559"
@@
 		(dnp no)
 		(fields_autoplaced yes)
-		(property "Reference" "D2"
+		(property "Reference" "D?"
 			(at 172.72 48.26 0)
 			(effects
@@
 		)
 		(instances
+			(project "Main"
+				(path "/77f264da-4c84-4b0c-9d20-4392731765e6/8078826c-4446-4e50-a209-45fcf7cbe7e4"
+					(reference "D?")
+					(unit 1)
+				)
+			)
 			(project "Power"
 				(path "/7fd1e59d-d896-4263-8d21-df7365fed559"
@@
 		(dnp no)
 		(fields_autoplaced yes)
-		(property "Reference" "R2"
+		(property "Reference" "R?"
 			(at 128.27 53.3399 0)
 			(effects
@@
 		)
 		(instances
+			(project "Main"
+				(path "/77f264da-4c84-4b0c-9d20-4392731765e6/8078826c-4446-4e50-a209-45fcf7cbe7e4"
+					(reference "R?")
+					(unit 1)
+				)
+			)
 			(project "Power"
 				(path "/7fd1e59d-d896-4263-8d21-df7365fed559"
@@
 		(dnp no)
 		(fields_autoplaced yes)
-		(property "Reference" "L1"
+		(property "Reference" "L?"
 			(at 116.84 21.59 90)
 			(effects
@@
 		)
 		(instances
+			(project "Main"
+				(path "/77f264da-4c84-4b0c-9d20-4392731765e6/8078826c-4446-4e50-a209-45fcf7cbe7e4"
+					(reference "L?")
+					(unit 1)
+				)
+			)
 			(project ""
 				(path "/7fd1e59d-d896-4263-8d21-df7365fed559"
@@
 		(dnp no)
 		(fields_autoplaced yes)
-		(property "Reference" "D5"
+		(property "Reference" "D?"
 			(at 144.78 78.74 0)
 			(effects
@@
 		)
 		(instances
+			(project "Main"
+				(path "/77f264da-4c84-4b0c-9d20-4392731765e6/8078826c-4446-4e50-a209-45fcf7cbe7e4"
+					(reference "D?")
+					(unit 1)
+				)
+			)
 			(project "Power"
 				(path "/7fd1e59d-d896-4263-8d21-df7365fed559"
@@
 		(dnp no)
 		(fields_autoplaced yes)
-		(property "Reference" "R?"
+		(property "Reference" "R7"
 			(at 198.12 33.0199 0)
 			(effects
@@
 		(dnp no)
 		(fields_autoplaced yes)
-		(property "Reference" "D1"
+		(property "Reference" "D?"
 			(at 110.49 36.8299 90)
 			(effects
@@
 		)
 		(instances
+			(project "Main"
+				(path "/77f264da-4c84-4b0c-9d20-4392731765e6/8078826c-4446-4e50-a209-45fcf7cbe7e4"
+					(reference "D?")
+					(unit 1)
+				)
+			)
 			(project ""
 				(path "/7fd1e59d-d896-4263-8d21-df7365fed559"
@@
 		(dnp no)
 		(fields_autoplaced yes)
-		(property "Reference" "D?"
+		(property "Reference" "D1"
 			(at 50.8 20.32 0)
 			(effects
@@
 		(dnp no)
 		(fields_autoplaced yes)
-		(property "Reference" "D3"
+		(property "Reference" "D?"
 			(at 172.72 36.83 0)
 			(effects
@@
 		)
 		(instances
+			(project "Main"
+				(path "/77f264da-4c84-4b0c-9d20-4392731765e6/8078826c-4446-4e50-a209-45fcf7cbe7e4"
+					(reference "D?")
+					(unit 1)
+				)
+			)
 			(project "Power"
 				(path "/7fd1e59d-d896-4263-8d21-df7365fed559"
@@
 		(dnp no)
 		(fields_autoplaced yes)
-		(property "Reference" "R?"
+		(property "Reference" "R8"
 			(at 198.12 43.1799 0)
 			(effects
@@
 		(dnp no)
 		(fields_autoplaced yes)
-		(property "Reference" "R?"
+		(property "Reference" "R9"
 			(at 182.88 48.26 90)
 			(effects
@@
 		(dnp no)
 		(fields_autoplaced yes)
-		(property "Reference" "C2"
+		(property "Reference" "C?"
 			(at 140.97 43.5609 0)
 			(effects
@@
 		)
 		(instances
+			(project "Main"
+				(path "/77f264da-4c84-4b0c-9d20-4392731765e6/8078826c-4446-4e50-a209-45fcf7cbe7e4"
+					(reference "C?")
+					(unit 1)
+				)
+			)
 			(project "Power"
 				(path "/7fd1e59d-d896-4263-8d21-df7365fed559"
@@
 		(dnp no)
 		(fields_autoplaced yes)
-		(property "Reference" "R1"
+		(property "Reference" "R?"
 			(at 128.27 36.8299 0)
 			(effects
@@
 		)
 		(instances
+			(project "Main"
+				(path "/77f264da-4c84-4b0c-9d20-4392731765e6/8078826c-4446-4e50-a209-45fcf7cbe7e4"
+					(reference "R?")
+					(unit 1)
+				)
+			)
 			(project ""
 				(path "/7fd1e59d-d896-4263-8d21-df7365fed559"
@@
 		(dnp no)
 		(fields_autoplaced yes)
-		(property "Reference" "U1"
+		(property "Reference" "U?"
 			(at 90.17 19.05 0)
 			(effects
@@
 		)
 		(instances
+			(project "Main"
+				(path "/77f264da-4c84-4b0c-9d20-4392731765e6/8078826c-4446-4e50-a209-45fcf7cbe7e4"
+					(reference "U?")
+					(unit 1)
+				)
+			)
 			(project ""
 				(path "/7fd1e59d-d896-4263-8d21-df7365fed559"
@@
 		(dnp no)
 		(fields_autoplaced yes)
-		(property "Reference" "C1"
+		(property "Reference" "C?"
 			(at 63.5 43.5609 0)
 			(effects
@@
 		)
 		(instances
+			(project "Main"
+				(path "/77f264da-4c84-4b0c-9d20-4392731765e6/8078826c-4446-4e50-a209-45fcf7cbe7e4"
+					(reference "C?")
+					(unit 1)
+				)
+			)
 			(project ""
 				(path "/7fd1e59d-d896-4263-8d21-df7365fed559"
@@
 		(dnp no)
 		(fields_autoplaced yes)
-		(property "Reference" "Q?"
+		(property "Reference" "Q1"
 			(at 209.55 20.32 90)
 			(effects
@@
 		(dnp no)
 		(fields_autoplaced yes)
-		(property "Reference" "D4"
+		(property "Reference" "D?"
 			(at 144.78 20.32 0)
 			(effects
@@
 		)
 		(instances
+			(project "Main"
+				(path "/77f264da-4c84-4b0c-9d20-4392731765e6/8078826c-4446-4e50-a209-45fcf7cbe7e4"
+					(reference "D?")
+					(unit 1)
+				)
+			)
 			(project "Power"
 				(path "/7fd1e59d-d896-4263-8d21-df7365fed559"
@@
 		(dnp no)
 		(fields_autoplaced yes)
-		(property "Reference" "J?"
+		(property "Reference" "J1"
 			(at 38.1 20.32 0)
 			(effects

Commit message: update
Parts:
- added J2: PIR, symbol Connector:Screw_Terminal_01x02
Connections:
- net PIR_MOUV is gone; now on net PWR_U/D: D?.2 (A)
- net GND: now also J2.1 (Pin_1)
- net PWR_U/D: no longer D?.2 (A)
- new net: D?.2 (A), J2.2 (Pin_2)
Other:
- moved on the sheet: D?
Changed lines of the file:
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@@
+	)
+	(junction
+		(at 166.37 66.04)
+		(diameter 0)
+		(color 0 0 0 0)
 	)
 	(junction
@@
 	(wire
 		(pts
+			(xy 163.83 57.15) (xy 166.37 57.15)
+		)
+		(stroke
+			(width 0)
+			(type default)
+		)
+	)
+	(wire
+		(pts
 			(xy 43.18 29.21) (xy 45.72 29.21)
 		)
@@
 	(wire
 		(pts
-			(xy 148.59 85.09) (xy 149.86 85.09)
+			(xy 148.59 93.98) (xy 149.86 93.98)
 		)
 		(stroke
@@
 	(wire
 		(pts
+			(xy 166.37 57.15) (xy 166.37 66.04)
+		)
+		(stroke
+			(width 0)
+			(type default)
+		)
+	)
+	(wire
+		(pts
+			(xy 165.1 43.18) (xy 168.91 43.18)
+		)
+		(stroke
+			(width 0)
+			(type default)
+		)
+	)
+	(wire
+		(pts
 			(xy 204.47 26.67) (xy 195.58 26.67)
 		)
@@
 	(wire
 		(pts
-			(xy 163.83 43.18) (xy 168.91 43.18)
-		)
-		(stroke
-			(width 0)
-			(type default)
-		)
-	)
-	(wire
-		(pts
 			(xy 100.33 31.75) (xy 102.87 31.75)
 		)
@@
 	(wire
 		(pts
-			(xy 137.16 66.04) (xy 195.58 66.04)
-		)
-		(stroke
-			(width 0)
-			(type default)
-		)
-	)
-	(wire
-		(pts
 			(xy 217.17 66.04) (xy 195.58 66.04)
 		)
@@
 	(wire
 		(pts
+			(xy 137.16 66.04) (xy 166.37 66.04)
+		)
+		(stroke
+			(width 0)
+			(type default)
+		)
+	)
+	(wire
+		(pts
 			(xy 125.73 41.91) (xy 125.73 45.72)
 		)
@@
 	(wire
 		(pts
-			(xy 149.86 26.67) (xy 149.86 85.09)
+			(xy 166.37 66.04) (xy 195.58 66.04)
+		)
+		(stroke
+			(width 0)
+			(type default)
+		)
+	)
+	(wire
+		(pts
+			(xy 149.86 26.67) (xy 149.86 93.98)
 		)
 		(stroke
@@
 		)
 	)
-	(hierarchical_label "PIR_MOUV"
+	(hierarchical_label "PWR_U{slash}D"
 		(shape input)
-		(at 163.83 43.18 180)
+		(at 165.1 43.18 180)
 		(effects
 			(font
@@
 		(shape input)
 		(at 41.91 66.04 180)
-		(effects
-			(font
-				(size 1.27 1.27)
-			)
-			(justify right)
-		)
-	)
-	(hierarchical_label "PWR_U{slash}D"
-		(shape input)
-		(at 163.83 54.61 180)
 		(effects
 			(font
@@
 	(symbol
 		(lib_id "Device:D")
-		(at 144.78 85.09 180)
+		(at 144.78 93.98 180)
 		(unit 1)
 		(exclude_from_sim no)
@@
 		(fields_autoplaced yes)
 		(property "Reference" "D?"
-			(at 144.78 78.74 0)
+			(at 144.78 87.63 0)
 			(effects
 				(font
@@
 		)
 		(property "Value" "D"
-			(at 144.78 81.28 0)
+			(at 144.78 90.17 0)
 			(effects
 				(font
@@
 		)
 		(property "Footprint" ""
-			(at 144.78 85.09 0)
+			(at 144.78 93.98 0)
 			(effects
 				(font
@@
 		)
 		(property "Datasheet" "~"
-			(at 144.78 85.09 0)
+			(at 144.78 93.98 0)
 			(effects
 				(font
@@
 		)
 		(property "Description" "Diode"
-			(at 144.78 85.09 0)
+			(at 144.78 93.98 0)
 			(effects
 				(font
@@
 		)
 		(property "Sim.Device" "D"
-			(at 144.78 85.09 0)
+			(at 144.78 93.98 0)
 			(effects
 				(font
@@
 		)
 		(property "Sim.Pins" "1=K 2=A"
-			(at 144.78 85.09 0)
+			(at 144.78 93.98 0)
 			(effects
 				(font
@@
 					(unit 1)
 				)
+			)
+		)
+	)
+	(symbol
+		(lib_id "Connector:Screw_Terminal_01x02")
+		(at 158.75 57.15 180)
+		(unit 1)
+		(exclude_from_sim no)
+		(in_bom yes)
+		(on_board yes)
+		(dnp no)
+		(fields_autoplaced yes)
+		(property "Reference" "J2"
+			(at 158.75 48.26 0)
+			(effects
+				(font
+					(size 1.27 1.27)
+				)
+			)
+		)
+		(property "Value" "PIR"
+			(at 158.75 50.8 0)
+			(effects
+				(font
+					(size 1.27 1.27)
+				)
+			)
+		)
+		(property "Footprint" ""
+			(at 158.75 57.15 0)
+			(effects
+				(font
+					(size 1.27 1.27)
+				)
+				(hide yes)
+			)
+		)
+		(property "Datasheet" "~"
+			(at 158.75 57.15 0)
+			(effects
+				(font
+					(size 1.27 1.27)
+				)
+				(hide yes)
+			)
+		)
+		(property "Description" "Generic screw terminal, single row, 01x02, script generated (kicad-library-utils/schlib/autogen/connector/)"
+			(at 158.75 57.15 0)
+			(effects
+				(font
+					(size 1.27 1.27)
+				)
+				(hide yes)
+			)
+		)
+		(pin "2"
+		)
+		(pin "1"
+		)
+		(instances
+			(project "Main"
+				(path "/77f264da-4c84-4b0c-9d20-4392731765e6/8078826c-4446-4e50-a209-45fcf7cbe7e4"
+					(reference "J2")
+					(unit 1)
+				)

Commit message: Update_07_01_2026
Parts:
- removed D?: D, symbol Device:D
- removed J2: PIR, symbol Connector:Screw_Terminal_01x02
- added U3: MIC2253, Package_DFN_QFN:DFN-12-1EP_3x3mm_P0.5mm_EP1.6x2.5mm_ThermalVias, symbol Regulator_Switching:MIC2253
Connections:
- net WAKE_UP: now reaches Q2.2 (B), R9.2
- net PIR_MOUV: now reaches D?.2 (A)
- new net: U3.13 (PGND), U3.5 (PGND), U3.6 (PGND)
- new net: U3.7 (SW), U3.8 (SW)
Other:
- moved on the sheet: D?, R9

Commit message: Update_She
Parts:
- removed C?: 220u, symbol Device:C_Polarized
- removed D? (x3): D, symbol Device:D
- removed Q2: NPN, symbol Simulation_SPICE:NPN
- removed U3: MIC2253, Package_DFN_QFN:DFN-12-1EP_3x3mm_P0.5mm_EP1.6x2.5mm_ThermalVias, symbol Regulator_Switching:MIC2253
- added C10, C9: 100nF, symbol Device:C
- added C11, C12, C5, C6, C7, C8: 220u, symbol Device:C_Polarized
- added D2, D3, D6: PMEG2010AEH, Diode_SMD:D_SOD-123F, symbol Diode:PMEG2010AEH
- added D4, D5: 1N4001, Diode_THT:D_DO-41_SOD81_P10.16mm_Horizontal, symbol Diode:1N4001
- added D7: 5V, symbol Device:D_Zener
- added J7: 1.8 - 5.5 - Battery, symbol Connector:Screw_Terminal_01x02
- added J8: Panneau, symbol Connector:Screw_Terminal_01x02
- added L1, L2: 68u, symbol Device:L
- added Q2, Q6: PN2222A, Package_TO_SOT_THT:TO-92_Inline, symbol Transistor_BJT:PN2222A
- added R10, R12: 10k, symbol Device:R_US
- added R11: 100k, symbol Device:R_US
- added R13, R14, R16: R_US, symbol Device:R_US
- added R15, R17: 1k, symbol Device:R_US
- added U3: MCP1662-xOT, Package_TO_SOT_SMD:SOT-23-5, symbol Driver_LED:MCP1662-xOT
- added U4: TPS63000, Package_SON:Texas_DRC0010J_ThermalVias, symbol Regulator_Switching:TPS63000
- added U5: MCP73831-2-OT, Package_TO_SOT_SMD:SOT-23-5, symbol Battery_Management:MCP73831-2-OT
- R7: value 100k -> 10k; footprint Resistor_SMD:R_0805_2012Metric_Pad1.20x1.40mm_HandSolder -> (none)
- R8: value 10k -> 2k; footprint Resistor_SMD:R_0805_2012Metric_Pad1.20x1.40mm_HandSolder -> (none)
- R9: value 1k -> 100k; footprint Resistor_SMD:R_0805_2012Metric_Pad1.20x1.40mm_HandSolder -> (none)
Connections:
- net +3.3V_BATT: now also Q1.3 (S), C10.2, D3.1 (K), D6.1 (K), R11.1; no longer Q1.1 (D), R7.1
- net +3.3V_POWER_UP: now also Q1.1 (D), R7.1, R9.1, C9.1, L1.1, U3.5 (V_{IN}); no longer Q1.3 (S)
- net 12V_POWER_UP: now also C5.1, D2.1 (K), R13.1
- net GND: now also R7.2, R8.2, C11.2, C12.2, C5.2, C6.2, C7.2, C8.2, C9.2, D7.2 (A), J7.1 (Pin_1), J8.1 (Pin_1), Q2.1 (E), Q6.1 (E), R14.2, U3.2 (GND), U4.11 (PGND), U4.3 (PGND), U4.9 (GND), U5.2 (V_{SS})
- net PIR_MOUV: now also D5.2 (A)
- net PWR_U/D: now also D4.2 (A)
- net at C?.1, L?.2, R?.1: now also D6.2 (A)
- net WAKE_UP: no longer names the net of R9.2
- net WAKE_UP: now also R10.1, U3.4 (EN)
- new net: D4.1 (K), D5.1 (K), R17.1
- new net: Q6.2 (B), R17.2
- new net: C10.1, Q1.2 (G), R11.2, R12.1
- new net: Q2.3 (C), R10.2
- new net: C11.1, D7.1 (K), J8.2 (Pin_2), U5.4 (V_{DD})
- new net: R8.1, U5.5 (PROG)
- new net: C6.1, C7.1, D3.2 (A), U4.1 (VOUT), U4.10 (FB)
- new net: D2.2 (A), L1.2, U3.1 (SW)
- new net: Q2.2 (B), R15.1
- new net: L2.1, U4.2 (L2)
- new net: L2.2, U4.4 (L1)
- new net: C8.1, R16.2, U4.6 (EN), U4.7 (PS/SYNC), U4.8 (VINA)
- new net: R13.2, R14.1, U3.3 (V_{FB})
- new net: Q6.3 (C), R12.2
- new net 12V_EN: R15.2
- new net RECHARGE_INFO: U5.1 (STAT)
- new net VOLTAGE_BAT: C12.1, J7.2 (Pin_2), R16.1, U4.5 (VIN), U5.3 (V_{BAT})
Other:
- moved on the sheet: C?, D1, D?, J1, L?, R?, U?
