File: Architecture/Main/Sensors.kicad_sch (KiCad schematic)
At the start: 0 parts

Commit message: Archi_1
Parts:
- added J6: Conn_01x04, symbol Connector_Generic:Conn_01x04
- added R5: LDR03, OptoDevice:R_LDR_10x8.5mm_P7.6mm_Vertical, symbol Sensor_Optical:LDR03
- added R6: 10k, symbol Device:R_US
Connections:
- net +3.3V: now also J6.1 (Pin_1), R5.1
- net GND: now also J6.4 (Pin_4), R6.2
- new net D36: R5.2, R6.1
- new net RX0: J6.3 (Pin_3)
- new net TX0: J6.2 (Pin_2)
Other:
- note added: "Brightness Sensor ( I/O D36 )"
- note added: "GND"
- note added: "GPS Sensor ( RX/TX0 )"
- note added: "RX_GPS"
- note added: "TX_GPS"
- note added: "VCC_GPS"

Commit message: Archi_2
Parts:
- added J4: Conn_01x04, symbol Connector_Generic:Conn_01x04
Connections:
- net +3.3V: now also J4.1 (Pin_1)
- net GND: now also J4.4 (Pin_4)
- new net DATA_DHT22: J4.2 (Pin_2)
- no-connect marks 0 -> 1
Other:
- note added: "DATA"
- note added: "DHT22 Sensor"
- note added: "NC"
- note added: "VCC"

Commit message: Update Schematic
Parts:
- added J2: Screw_Terminal_01x02, symbol Connector:Screw_Terminal_01x02
Connections:
- net GND: now also J2.2 (Pin_2)
- net MOUV: now also J2.1 (Pin_1)
Other:
- note added: "PIR - Mouvement Sensor"
- note removed: "PINOUT"

Commit message: Update
Connections:
- net D36 renamed BRIGHTNESS_SENSOR
Changed lines of the file:
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@@
 	)
 	(rectangle
-		(start 203.2 25.4)
+		(start 189.23 25.4)
 		(end 266.7 63.5)
 		(stroke
@@
 		)
 	)
+	(hierarchical_label "I2C_SCL"
+		(shape input)
+		(at 74.93 50.8 0)
+		(effects
+			(font
+				(size 1.27 1.27)
+			)
+			(justify left)
+		)
+	)
 	(hierarchical_label "MOUV"
 		(shape input)
@@
 		)
 	)
-	(hierarchical_label "D36"
+	(hierarchical_label "BRIGHTNESS_SENSOR"
 		(shape input)
 		(at 213.36 43.18 180)
@@
 		)
 	)
+	(hierarchical_label "I2C_SDA"
+		(shape input)
+		(at 74.93 46.99 0)
+		(effects
+			(font
+				(size 1.27 1.27)
+			)
+			(justify left)
+		)
+	)

Commit message: update
Parts:
- removed J2: Screw_Terminal_01x02, symbol Connector:Screw_Terminal_01x02
Other:
- note removed: "PIR - Mouvement Sensor"
- moved on the sheet: J4, J6, R5, R6

Commit message: Update_07_01_2026
Parts:
- added C2, C3: 100nF, symbol Device:C
- added J3: Conn_01x03, symbol Connector_Generic:Conn_01x03
- R5, R6: now not fitted; now left out of the parts list
Connections:
- net +3.3V: now also C2.1, C3.1
- net GND: now also C2.2, C3.2, J3.3 (Pin_3)
- new net +3.3V_BATTERY: J3.1 (Pin_1)
- new net PIR_MOUV: J3.2 (Pin_2)
Other:
- moved on the sheet: J4, J6

Commit message: CodeFinalProto_plus_majarchitecture
Parts:
- added R3, R4: 10k, symbol Device:R_US
Connections:
- net +3.3V_BATTERY: now also R3.1
- net GND: now also R4.2
- new net Voltage_Batt: R3.2, R4.1
Other:
- note added: "Battery Voltage"
- note added: "PIR - Mouv Detector"

Commit message: Update_She
Connections:
- net +3.3V_BATTERY: no longer R3.1
- net Voltage_Batt: now also R3.1; no longer R3.2, R4.1
- new net Voltage_Batt_value: R3.2, R4.1
Changed lines of the file:
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@@
-		)
-	)
-	(hierarchical_label "+3.3V_BATTERY"
-		(shape input)
-		(at 44.45 78.74 180)
-		(effects
-			(font
-				(size 1.27 1.27)
-			)
-			(justify right)
 		)
 	)
@@
 		)
 	)
-	(hierarchical_label "Voltage_Batt"
+	(hierarchical_label "Voltage_Batt_value"
 		(shape input)
 		(at 44.45 91.44 180)
@@
 		(effects
 			(font
+				(size 1.27 1.27)
+			)
+			(justify right)
+		)
+	)
+	(hierarchical_label "Voltage_Batt"
+		(shape input)
+		(at 44.45 78.74 180)
+		(effects
+			(font
