File: Architecture/Main-REVA2/uc.kicad_sch (KiCad schematic)
At the start: 3 parts

Commit message: Update_Schematic
Connections:
- net +3V3 is gone; now on net VIN: R18.2, R19.2, U6. (GND)
- new net +3.3V: U6. (GND)
Other:
- company: (none) -> Polytech Nantes - ETN4
- title: (none) -> Collecteur de données Animalières
Changed lines of the file:
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@@
 	(generator_version "9.0")
 	(paper "A4")
+	(title_block
+		(title "Collecteur de données Animalières")
+		(date "2025-11-28")
+		(rev "A2")
+		(company "Polytech Nantes - ETN4")
+		(comment 1 "Architecture Collectuer de données")
+		(comment 2 "Brain Page")
+	)
 	(text "#ifndef __CONFIG_H__\n#define __CONFIG_H__\n\n// --- SYSTÈME (LIAISON PC) ---\n// Note : Pour libérer 43/44, utilisez l'USB natif sur GPIO 19/20\n// Dans PlatformIO : build_flags = -DARDUINO_USB_CDC_ON_BOOT=1\n\n// --- MODULE 4G LTE (UART1 ou UART0 réassigné) ---\n#define MODEM_RX          43  \n#define MODEM_TX          44  \n\n// --- GPS EXTERNE (UART2) ---\n#define GPS_RX_PIN        16 \n#define GPS_TX_PIN        17 \n\n// --- CARTE SD (SPI) ---\n#define SD_SCK            14 \n#define SD_MISO           12 \n#define SD_MOSI           13 \n#define SD_CS             15 \n\n// --- CAMERA PINS (SÉCURISÉ POUR N16R8) ---\n#define SIOD_GPIO_NUM     21 \n#define SIOC_GPIO_NUM     22 \n#define XCLK_GPIO         -1  \n#define PCLK_GPIO         46  \n#define VSYNC_GPIO        3   \n#define HREF_GPIO         25 \n#define D0_GPIO           26 \n#define D1_GPIO           47  \n#define D2_GPIO           39 \n#define D3_GPIO           32 \n#define D4_GPIO           27 \n#define D5_GPIO           23 \n#define D6_GPIO           45   // Déplacé depuis 20 pour laisser le port USB Natif libre\n#define D7_GPIO           18 \n\n// --- PINS LIBRES ---\n#define FREE_GPIO_0       0\n#define FREE_GPIO_6       6\n#define FREE_GPIO_7       7\n#define FREE_GPIO_8       8\n#define FREE_GPIO_9       9\n#define FREE_GPIO_10      10\n#define FREE_GPIO_11      11\n#define FREE_GPIO_20      20   // Réservé USB Natif (D+)\n#define FREE_GPIO_48      48\n\n// --- PINS INTERDITES (PSRAM/FLASH) ---\n// GPIO 19, 28-31, 33-37\n#endif"
 		(exclude_from_sim no)
-		(at 215.646 72.39 0)
+		(at 209.55 98.298 0)
 		(effects
 			(font
@@
 	(wire
 		(pts
-			(xy 92.71 29.21) (xy 92.71 27.94)
-		)
-		(stroke
-			(width 0)
-			(type default)
-		)
-	)
-	(wire
-		(pts
 			(xy 130.81 59.69) (xy 133.35 59.69)
 		)
@@
 		)
 	)
+	(hierarchical_label "VIN"
+		(shape input)
+		(at 83.82 45.72 90)
+		(effects
+			(font
+				(size 1.27 1.27)
+			)
+			(justify left)
+		)
+	)
 	(hierarchical_label "D4"
 		(shape input)
@@
 		)
 	)
+	(hierarchical_label "VIN"
+		(shape input)
+		(at 74.93 45.72 90)
+		(effects
+			(font
+				(size 1.27 1.27)
+			)
+			(justify left)
+		)
+	)
 	(hierarchical_label "D1"
 		(shape input)
@@
 	)
 	(symbol
-		(lib_id "power:+3V3")
-		(at 74.93 45.72 0)
-		(unit 1)
-		(exclude_from_sim no)
-		(in_bom yes)
-		(on_board yes)
-		(dnp no)
-		(fields_autoplaced yes)
-		(property "Reference" "#PWR08"
-			(at 74.93 49.53 0)
-			(effects
-				(font
-					(size 1.27 1.27)
-				)
-				(hide yes)
-			)
-		)
-		(property "Value" "+3V3"
-			(at 74.93 40.64 0)
-			(effects
-				(font
-					(size 1.27 1.27)
-				)
-			)
-		)
-		(property "Footprint" ""
-			(at 74.93 45.72 0)
-			(effects
-				(font
-					(size 1.27 1.27)
-				)
-				(hide yes)
-			)
-		)
-		(property "Datasheet" ""
-			(at 74.93 45.72 0)
-			(effects
-				(font
-					(size 1.27 1.27)
-				)
-				(hide yes)
-			)
-		)
-		(property "Description" "Power symbol creates a global label with name \"+3V3\""
-			(at 74.93 45.72 0)
-			(effects
-				(font
-					(size 1.27 1.27)
-				)
-				(hide yes)
-			)
-		)
-		(pin "1"
-		)
-		(instances
-			(project "Main"
-				(path "/77f264da-4c84-4b0c-9d20-4392731765e6/663cc000-5ebd-47ff-83ef-c87f1fdc0c98"
-					(reference "#PWR08")
-					(unit 1)
-				)
-			)
-		)
-	)
-	(symbol
-		(lib_id "power:+3V3")
-		(at 92.71 27.94 0)
-		(unit 1)
-		(exclude_from_sim no)
-		(in_bom yes)
-		(on_board yes)
-		(dnp no)
-		(fields_autoplaced yes)
-		(property "Reference" "#PWR012"
-			(at 92.71 31.75 0)
-			(effects
-				(font
-					(size 1.27 1.27)
-				)
-				(hide yes)
-			)
-		)
-		(property "Value" "+3V3"
-			(at 92.71 22.86 0)
-			(effects
-				(font
-					(size 1.27 1.27)
-				)
-			)
-		)
-		(property "Footprint" ""
-			(at 92.71 27.94 0)
-			(effects
-				(font
-					(size 1.27 1.27)
-				)
-				(hide yes)
-			)
-		)
-		(property "Datasheet" ""
-			(at 92.71 27.94 0)
-			(effects
-				(font
-					(size 1.27 1.27)
-				)
-				(hide yes)
-			)
-		)
-		(property "Description" "Power symbol creates a global label with name \"+3V3\""
-			(at 92.71 27.94 0)
-			(effects
-				(font
-					(size 1.27 1.27)
-				)
-				(hide yes)
-			)
-		)
-		(pin "1"
-		)
-		(instances
-			(project "Main"
-				(path "/77f264da-4c84-4b0c-9d20-4392731765e6/663cc000-5ebd-47ff-83ef-c87f1fdc0c98"
-					(reference "#PWR012")
-					(unit 1)
-				)
-			)
-		)
-	)
-	(symbol
 		(lib_id "Device:R_US")
 		(at 74.93 50.8 180)
@@
 					(unit 1)
 				)
-			)
-		)
-	)
-	(symbol
-		(lib_id "power:+3V3")
-		(at 83.82 45.72 0)
-		(unit 1)
-		(exclude_from_sim no)
-		(in_bom yes)
-		(on_board yes)
-		(dnp no)
-		(fields_autoplaced yes)
-		(property "Reference" "#PWR09"
-			(at 83.82 49.53 0)
-			(effects
-				(font
-					(size 1.27 1.27)
-				)
-				(hide yes)
-			)
-		)
-		(property "Value" "+3V3"
-			(at 83.82 40.64 0)
-			(effects
-				(font
-					(size 1.27 1.27)
-				)
-			)
-		)
-		(property "Footprint" ""
-			(at 83.82 45.72 0)
-			(effects
-				(font
-					(size 1.27 1.27)
-				)
-				(hide yes)
-			)
-		)
-		(property "Datasheet" ""
-			(at 83.82 45.72 0)
-			(effects
-				(font
-					(size 1.27 1.27)
-				)
-				(hide yes)
-			)
-		)
-		(property "Description" "Power symbol creates a global label with name \"+3V3\""
-			(at 83.82 45.72 0)
-			(effects
-				(font
-					(size 1.27 1.27)
-				)
-				(hide yes)
-			)
-		)
-		(pin "1"
-		)
-		(instances
-			(project "Main"
-				(path "/77f264da-4c84-4b0c-9d20-4392731765e6/663cc000-5ebd-47ff-83ef-c87f1fdc0c98"
-					(reference "#PWR09")
-					(unit 1)
-				)

Commit message: Update
Parts:
- removed U6: ~, symbol MCU:ESP32-S3-N16R8
- added U4: ESP32-S3-DEVKITC-1-N8R8, CollecteurDonne:ESP32-S3-DEVKITC-1-N8R8, symbol ESP32-S3-DEVKITC-1-N8R8:ESP32-S3-DEVKITC-1-N8R8
Connections:
- net +3.3V: now also U4.J1_1 (3V3), U4.J1_2 (3V3.)
- net CLK: now also U4.J1_19 (GPIO13)
- net CS: now also U4.J1_16 (GPIO10)
- net D1: now also U4.J3_4 (GPIO1)
- net D14: now also U4.J1_20 (GPIO14)
- net D15: now also U4.J1_8 (GPIO15)
- net D18: now also U4.J1_11 (GPIO18)
- net D2: now also U4.J3_5 (GPIO2)
- net D21: now also U4.J3_18 (GPIO21)
- net D3: now also U4.J1_13 (GPIO3)
- net D39: now also U4.J3_10 (GPIO38), U4.J3_9 (MTCK/GPIO39)
- net D4: now also U4.J1_4 (GPIO4)
- net D40: now also U4.J3_8 (MTDO/GPIO40)
- net D45: now also U4.J3_15 (GPIO45)
- net D46: now also U4.J1_14 (GPIO46)
- net D47: now also U4.J3_17 (GPIO47)
- net D48: now also U4.J3_16 (GPIO48)
- net D5: now also U4.J1_5 (GPIO5)
- net D6: now also U4.J1_6 (GPIO6)
- net D7: now also U4.J1_7 (GPIO7)
- net GND: now also U4.J1_22 (GND3), U4.J3_1 (GND), U4.J3_21 (GND1), U4.J3_22 (GND2)
- net I2C_SCL: now also U4.J1_15 (GPIO9)
- net I2C_SDA: now also U4.J1_12 (GPIO8)
- net MISO: now also U4.J1_18 (GPIO12)
- net MOSI: now also U4.J1_17 (GPIO11)
- net RX1: now also U4.J1_10 (GPIO17)
- net RX2: now also U4.J3_7 (MTDI/GPIO41)
- net TX1: now also U4.J1_9 (GPIO16)
- net TX2: now also U4.J3_6 (MTMS/GPIO42)
- net VIN: now also U4.J1_21 (5V0)
Other:
- moved on the sheet: R18, R19

Commit message: Update_Sche
Parts:
- R18, R19: footprint (none) -> CollecteurDonne:Résistance L10mm
Changed lines of the file:
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@@
 			)
 		)
-		(property "Footprint" ""
+		(property "Footprint" "CollecteurDonne:Résistance L10mm"
 			(at 72.644 54.356 90)
 			(effects
@@
 			)
 		)
-		(property "Footprint" ""
+		(property "Footprint" "CollecteurDonne:Résistance L10mm"
 			(at 63.754 54.356 90)
 			(effects

Commit message: Update_Schematic_PCB
Parts:
- added C20: 100nF, CollecteurDonne:C_Disc_D5.0mm_W2.5mm_P5.00mm, symbol Device:C
- added D3: D, CollecteurDonne:D_DO-35_SOD27_P7.62mm_Horizontal, symbol Device:D
- R18, R19: footprint CollecteurDonne:Résistance L10mm -> CollecteurDonne:R_Axial_DIN0207_L6.3mm_D2.5mm_P10.16mm_Horizontal
Connections:
- net D18 is gone; now on net RX1: U4.J1_11 (GPIO18)
- net GND: now also C20.2
- net RX1: no longer U4.J1_10 (GPIO17)
- net TX1: now also U4.J1_10 (GPIO17); no longer U4.J1_9 (GPIO16)
- net VIN: now also D3.2 (A); no longer U4.J1_21 (5V0)
- new net: C20.1, D3.1 (K), U4.J1_21 (5V0)
- new net D16: U4.J1_9 (GPIO16)
Other:
- moved on the sheet: R18, R19, U4

Commit message: Update_28_01_2025
Connections:
- net D39: no longer U4.J3_10 (GPIO38)
- new net D38: U4.J3_10 (GPIO38)
Changed lines of the file:
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@@
 		)
 	)
-	(hierarchical_label "D39"
+	(hierarchical_label "D38"
 		(shape input)
 		(at 132.08 73.66 0)
