File: Architecture/Main-REVA2/uc.kicad_sch (KiCad schematic)
At the start: 5 parts, among them U4 ESP32-S3-DEVKITC-1-N8R8

Commit message: update_01_02_2026
Parts:
- added C18: 470uF, symbol Device:C_Polarized
Connections:
- net GND: now also C18.2
- net at C20.1, D3.1 (K), U4.J1_21 (5V0): now also C18.1
Other:
- moved on the sheet: D3
Changed lines of the file:
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@@
 	)
 	(junction
+		(at 52.07 101.6)
+		(diameter 0)
+		(color 0 0 0 0)
+	)
+	(junction
 		(at 81.28 101.6)
 		(diameter 0)
@@
 		(color 0 0 0 0)
 	)
+	(junction
+		(at 64.77 114.3)
+		(diameter 0)
+		(color 0 0 0 0)
+	)
 	(no_connect
 		(at 132.08 96.52)
@@
 	(wire
 		(pts
+			(xy 52.07 101.6) (xy 64.77 101.6)
+		)
+		(stroke
+			(width 0)
+			(type default)
+		)
+	)
+	(wire
+		(pts
 			(xy 129.54 99.06) (xy 132.08 99.06)
 		)
@@
 	(wire
 		(pts
-			(xy 49.53 101.6) (xy 53.34 101.6)
+			(xy 38.1 101.6) (xy 41.91 101.6)
 		)
 		(stroke
@@
 	(wire
 		(pts
+			(xy 52.07 101.6) (xy 52.07 104.14)
+		)
+		(stroke
+			(width 0)
+			(type default)
+		)
+	)
+	(wire
+		(pts
 			(xy 129.54 55.88) (xy 132.08 55.88)
 		)
@@
 	(wire
 		(pts
-			(xy 60.96 101.6) (xy 64.77 101.6)
+			(xy 49.53 101.6) (xy 52.07 101.6)
 		)
 		(stroke
@@
 	(wire
 		(pts
+			(xy 52.07 111.76) (xy 52.07 114.3)
+		)
+		(stroke
+			(width 0)
+			(type default)
+		)
+	)
+	(wire
+		(pts
 			(xy 81.28 58.42) (xy 83.82 58.42)
 		)
@@
 		)
 	)
+	(wire
+		(pts
+			(xy 52.07 114.3) (xy 64.77 114.3)
+		)
+		(stroke
+			(width 0)
+			(type default)
+		)
+	)
 	(image
 		(at 110.49 144.78)
@@
 	(hierarchical_label "VIN"
 		(shape input)
-		(at 49.53 101.6 180)
+		(at 38.1 101.6 180)
 		(effects
 			(font
@@
 	)
 	(symbol
+		(lib_id "Device:C_Polarized")
+		(at 52.07 107.95 0)
+		(unit 1)
+		(exclude_from_sim no)
+		(in_bom yes)
+		(on_board yes)
+		(dnp no)
+		(fields_autoplaced yes)
+		(property "Reference" "C18"
+			(at 55.88 105.7909 0)
+			(effects
+				(font
+					(size 1.27 1.27)
+				)
+				(justify left)
+			)
+		)
+		(property "Value" "470uF"
+			(at 55.88 108.3309 0)
+			(effects
+				(font
+					(size 1.27 1.27)
+				)
+				(justify left)
+			)
+		)
+		(property "Footprint" ""
+			(at 53.0352 111.76 0)
+			(effects
+				(font
+					(size 1.27 1.27)
+				)
+				(hide yes)
+			)
+		)
+		(property "Datasheet" "~"
+			(at 52.07 107.95 0)
+			(effects
+				(font
+					(size 1.27 1.27)
+				)
+				(hide yes)
+			)
+		)
+		(property "Description" "Polarized capacitor"
+			(at 52.07 107.95 0)
+			(effects
+				(font
+					(size 1.27 1.27)
+				)
+				(hide yes)
+			)
+		)
+		(pin "1"
+		)
+		(pin "2"
+		)
+		(instances
+			(project ""
+				(path "/77f264da-4c84-4b0c-9d20-4392731765e6/663cc000-5ebd-47ff-83ef-c87f1fdc0c98"
+					(reference "C18")
+					(unit 1)
+				)
+			)
+		)
+	)
+	(symbol
 		(lib_id "Device:C")
 		(at 64.77 107.95 0)
@@
 	(symbol
 		(lib_id "Device:D")
-		(at 57.15 101.6 180)
+		(at 45.72 101.6 180)
 		(unit 1)
 		(exclude_from_sim no)
@@
 		(dnp no)
 		(property "Reference" "D3"
-			(at 57.15 98.552 0)
+			(at 45.72 98.552 0)
 			(effects
 				(font
@@
 		)
 		(property "Value" "D"
-			(at 57.15 104.394 0)
+			(at 45.72 104.394 0)
 			(effects
 				(font
@@
 		)
 		(property "Footprint" "CollecteurDonne:D_DO-35_SOD27_P7.62mm_Horizontal"
-			(at 57.15 101.6 0)
+			(at 45.72 101.6 0)
 			(effects
 				(font
@@
 		)
 		(property "Datasheet" "~"
-			(at 57.15 101.6 0)
+			(at 45.72 101.6 0)
 			(effects
 				(font
@@
 		)
 		(property "Description" "Diode"
-			(at 57.15 101.6 0)
+			(at 45.72 101.6 0)
 			(effects
 				(font
@@
 		)
 		(property "Sim.Device" "D"
-			(at 57.15 101.6 0)
+			(at 45.72 101.6 0)
 			(effects
 				(font
@@
 		)
 		(property "Sim.Pins" "1=K 2=A"
-			(at 57.15 101.6 0)
+			(at 45.72 101.6 0)
 			(effects
 				(font

Commit message: Update_6_02_2026
Parts:
- C18: value 470uF -> 100uF; footprint (none) -> CollecteurDonne:C_Radial_D10.0mm_H16.0mm_P5.00mm
Changed lines of the file:
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@@
 			)
 		)
-		(property "Value" "470uF"
+		(property "Value" "100uF"
 			(at 55.88 108.3309 0)
 			(effects
@@
 			)
 		)
-		(property "Footprint" ""
+		(property "Footprint" "CollecteurDonne:C_Radial_D10.0mm_H16.0mm_P5.00mm"
 			(at 53.0352 111.76 0)
 			(effects

Commit message: Update
Other:
- note removed: "#ifndef __CONFIG_H__ #define __CONFIG_H__ // --- SYSTÈME (LIAISON PC) --- // Note : Pour libérer 43/44, utilisez l'USB natif sur GPIO 19/20 // Dans PlatformIO : build_flags = -DARDUINO_USB_CDC_ON_BOOT=1 // --- MODULE 4G LTE (UART1 ou UART0 réassigné) --- #define MODEM_RX 43 #define MODEM_TX 44 // --- GPS EXTERNE (UART2) --- #define GPS_RX_PIN 16 #define GPS_TX_PIN 17 // --- CARTE SD (SPI) --- #de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"
Changed lines of the file:
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@@
 		(comment 2 "Brain Page")
 	)
-	(text "#ifndef __CONFIG_H__\n#define __CONFIG_H__\n\n// --- SYSTÈME (LIAISON PC) ---\n// Note : Pour libérer 43/44, utilisez l'USB natif sur GPIO 19/20\n// Dans PlatformIO : build_flags = -DARDUINO_USB_CDC_ON_BOOT=1\n\n// --- MODULE 4G LTE (UART1 ou UART0 réassigné) ---\n#define MODEM_RX          43  \n#define MODEM_TX          44  \n\n// --- GPS EXTERNE (UART2) ---\n#define GPS_RX_PIN        16 \n#define GPS_TX_PIN        17 \n\n// --- CARTE SD (SPI) ---\n#define SD_SCK            14 \n#define SD_MISO           12 \n#define SD_MOSI           13 \n#define SD_CS             15 \n\n// --- CAMERA PINS (SÉCURISÉ POUR N16R8) ---\n#define SIOD_GPIO_NUM     21 \n#define SIOC_GPIO_NUM     22 \n#define XCLK_GPIO         -1  \n#define PCLK_GPIO         46  \n#define VSYNC_GPIO        3   \n#define HREF_GPIO         25 \n#define D0_GPIO           26 \n#define D1_GPIO           47  \n#define D2_GPIO           39 \n#define D3_GPIO           32 \n#define D4_GPIO           27 \n#define D5_GPIO           23 \n#define D6_GPIO           45   // Déplacé depuis 20 pour laisser le port USB Natif libre\n#define D7_GPIO           18 \n\n// --- PINS LIBRES ---\n#define FREE_GPIO_0       0\n#define FREE_GPIO_6       6\n#define FREE_GPIO_7       7\n#define FREE_GPIO_8       8\n#define FREE_GPIO_9       9\n#define FREE_GPIO_10      10\n#define FREE_GPIO_11      11\n#define FREE_GPIO_20      20   // Réservé USB Natif (D+)\n#define FREE_GPIO_48      48\n\n// --- PINS INTERDITES (PSRAM/FLASH) ---\n// GPIO 19, 28-31, 33-37\n#endif"
-		(exclude_from_sim no)
-		(at 209.55 98.298 0)
-		(effects
-			(font
-				(size 1.27 1.27)
-			)
-		)
-	)
 	(junction
 		(at 71.12 78.74)
@@
 		)
 		(stroke
+			(width 0)
+			(type default)
+		)
+	)
+	(wire
+		(pts
+			(xy 168.91 92.71) (xy 168.91 91.44)
+		)
+		(stroke

Commit message: Update_09_04_2026_PC
Other:
- moved on the sheet: C18, C20, D3, R18, R19, U4
