File: Architecture/Main-REVA2/Cam.kicad_sch (KiCad schematic)
At the start: 3 parts, among them J2 Conn_01x02

Commit message: Update_Schematic
Parts:
- added C7: 100nF, symbol Device:C
- gave numbers to parts that had none: 1
Connections:
- net 12V: now also C7.1
- net GND: now also C7.2
- net +3.3V renamed +VCC
Other:
- company: (none) -> Polytech Nantes - ETN4
- title: (none) -> Collecteur de données Animalières
Changed lines of the file:
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@@
 	(generator_version "9.0")
 	(paper "A4")
+	(title_block
+		(title "Collecteur de données Animalières")
+		(date "2025-11-28")
+		(rev "A2")
+		(company "Polytech Nantes - ETN4")
+		(comment 1 "Architecture Collectuer de données")
+		(comment 2 "Camera Page")
+	)
 	(rectangle
 		(start 139.7 92.71)
@@
 	)
 	(junction
+		(at 175.26 105.41)
+		(diameter 0)
+		(color 0 0 0 0)
+	)
+	(junction
+		(at 184.15 114.3)
+		(diameter 0)
+		(color 0 0 0 0)
+	)
+	(junction
 		(at 154.94 64.77)
 		(diameter 0)
@@
 	(wire
 		(pts
-			(xy 171.45 105.41) (xy 185.42 105.41)
+			(xy 171.45 105.41) (xy 175.26 105.41)
 		)
 		(stroke
@@
 	(wire
 		(pts
+			(xy 175.26 105.41) (xy 185.42 105.41)
+		)
+		(stroke
+			(width 0)
+			(type default)
+		)
+	)
+	(wire
+		(pts
+			(xy 175.26 114.3) (xy 184.15 114.3)
+		)
+		(stroke
+			(width 0)
+			(type default)
+		)
+	)
+	(wire
+		(pts
 			(xy 189.23 82.55) (xy 193.04 82.55)
 		)
@@
 	(wire
 		(pts
+			(xy 175.26 113.03) (xy 175.26 114.3)
+		)
+		(stroke
+			(width 0)
+			(type default)
+		)
+	)
+	(wire
+		(pts
 			(xy 154.94 64.77) (xy 176.53 64.77)
 		)
@@
 	(wire
 		(pts
-			(xy 184.15 107.95) (xy 184.15 111.76)
+			(xy 184.15 107.95) (xy 184.15 114.3)
 		)
 		(stroke
@@
 	(wire
 		(pts
+			(xy 184.15 116.84) (xy 184.15 114.3)
+		)
+		(stroke
+			(width 0)
+			(type default)
+		)
+	)
+	(wire
+		(pts
 			(xy 189.23 77.47) (xy 193.04 77.47)
 		)
@@
 		)
 	)
-	(hierarchical_label "PWDN"
-		(shape input)
-		(at 193.04 85.09 0)
-		(effects
-			(font
-				(size 1.27 1.27)
-			)
-			(justify left)
-		)
-	)
 	(hierarchical_label "D0"
 		(shape input)
@@
 		)
 	)
-	(hierarchical_label "+3.3V"
+	(hierarchical_label "PWDN"
+		(shape input)
+		(at 193.04 85.09 0)
+		(effects
+			(font
+				(size 1.27 1.27)
+			)
+			(justify left)
+		)
+	)
+	(hierarchical_label "+VCC"
 		(shape input)
 		(at 152.4 64.77 180)
@@
 	)
 	(symbol
+		(lib_id "Device:C")
+		(at 175.26 109.22 0)
+		(unit 1)
+		(exclude_from_sim no)
+		(in_bom yes)
+		(on_board yes)
+		(dnp no)
+		(property "Reference" "C7"
+			(at 166.624 110.998 0)
+			(effects
+				(font
+					(size 1.27 1.27)
+				)
+				(justify left)
+			)
+		)
+		(property "Value" "100nF"
+			(at 166.624 113.538 0)
+			(effects
+				(font
+					(size 1.27 1.27)
+				)
+				(justify left)
+			)
+		)
+		(property "Footprint" ""
+			(at 176.2252 113.03 0)
+			(effects
+				(font
+					(size 1.27 1.27)
+				)
+				(hide yes)
+			)
+		)
+		(property "Datasheet" "~"
+			(at 175.26 109.22 0)
+			(effects
+				(font
+					(size 1.27 1.27)
+				)
+				(hide yes)
+			)
+		)
+		(property "Description" "Unpolarized capacitor"
+			(at 175.26 109.22 0)
+			(effects
+				(font
+					(size 1.27 1.27)
+				)
+				(hide yes)
+			)
+		)
+		(pin "1"
+		)
+		(pin "2"
+		)
+		(instances
+			(project "Main"
+				(path "/77f264da-4c84-4b0c-9d20-4392731765e6/90e676b5-e192-40ef-8f2d-7a9315f03418"
+					(reference "C7")
+					(unit 1)
+				)
+			)
+		)
+	)
+	(symbol
 		(lib_id "Connector_Generic:Conn_01x02")
 		(at 190.5 105.41 0)
@@
 	(symbol
 		(lib_id "power:GND")
-		(at 184.15 111.76 0)
+		(at 184.15 116.84 0)
 		(unit 1)
 		(exclude_from_sim no)
@@
 		(fields_autoplaced yes)
 		(property "Reference" "#PWR024"
-			(at 184.15 118.11 0)
+			(at 184.15 123.19 0)
 			(effects
 				(font
@@
 		)
 		(property "Value" "GND"
-			(at 184.15 116.84 0)
+			(at 184.15 121.92 0)
 			(effects
 				(font
@@
 		)
 		(property "Footprint" ""
-			(at 184.15 111.76 0)
+			(at 184.15 116.84 0)
 			(effects
 				(font
@@
 		)
 		(property "Datasheet" ""
-			(at 184.15 111.76 0)
+			(at 184.15 116.84 0)
 			(effects
 				(font
@@
 		)
 		(property "Description" "Power symbol creates a global label with name \"GND\" , ground"
-			(at 184.15 111.76 0)
+			(at 184.15 116.84 0)
 			(effects
 				(font
@@
 		(dnp no)
 		(fields_autoplaced yes)
-		(property "Reference" "J?"
+		(property "Reference" "J11"
 			(at 182.88 58.42 0)
 			(effects
@@
 			(project "Main"
 				(path "/77f264da-4c84-4b0c-9d20-4392731765e6/90e676b5-e192-40ef-8f2d-7a9315f03418"
-					(reference "J?")
+					(reference "J11")
 					(unit 1)
 				)

Commit message: Update
Parts:
- removed J11: Conn_02x09_Counter_Clockwise, symbol Connector_Generic:Conn_02x09_Counter_Clockwise
- added H5, H6: MountingHole, MountingHole:MountingHole_3.2mm_M3_ISO14580, symbol Mechanical:MountingHole
- added U6: ~, symbol CollecteurDonneLIB:OV2640
- C1, C7: footprint (none) -> Capacitor_THT:C_Disc_D4.3mm_W1.9mm_P5.00mm; Fabricant (none) -> KEMET; Fournisseur (none) -> RS; Ref Fabricant (none) -> C0805C104K4RACTU; Ref Fournisseur (none) -> 648-0957
- J2: Fabricant (none) -> TE Connectivity; Fournisseur (none) -> RS; Ref Fabricant (none) -> 440054-2; Ref Fournisseur (none) -> 718-8526
Connections:
- net D0: now also U6.15
- net D1: now also U6.5
- net D2: now also U6.14
- net D3: now also U6.6
- net D4: now also U6.13
- net D5: now also U6.7
- net D6: now also U6.12
- net D7: now also U6.8
- net DCLK: now also U6.11
- net GND: now also U6.18
- net HREF: now also U6.3
- net PWDN: now also U6.10
- net RST: now also U6.4
- net SCL: now also U6.17
- net SDA: now also U6.16
- net VREF: now also U6.2
- net +VCC renamed +VCC_Alim
- net +VCC_Alim: now also U6.1
Other:
- note added: "https://fr.rs-online.com/web/p/borniers-enfichables/0446319"
- note added: "https://fr.rs-online.com/web/p/borniers-enfichables/0446488"
- moved on the sheet: C1, C7, J2

Commit message: Update_Sche
Parts:
- C1, C7: footprint Capacitor_THT:C_Disc_D4.3mm_W1.9mm_P5.00mm -> CollecteurDonne:Capa disc radial 5.08mm
- H5, H6: footprint MountingHole:MountingHole_3.2mm_M3_ISO14580 -> CollecteurDonne:MountingHole_2.2mm_M2_ISO7380
- J2: footprint (none) -> CollecteurDonne:ESP32-S3-DEVKITC-1-N8R8
- U6: footprint (none) -> Connector_PinSocket_1.27mm:PinSocket_2x09_P1.27mm_Vertical_SMD
Changed lines of the file:
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@@
 			)
 		)
-		(property "Footprint" "MountingHole:MountingHole_3.2mm_M3_ISO14580"
+		(property "Footprint" "CollecteurDonne:MountingHole_2.2mm_M2_ISO7380"
 			(at 248.92 35.56 0)
 			(effects
@@
 			)
 		)
-		(property "Footprint" ""
+		(property "Footprint" "Connector_PinSocket_1.27mm:PinSocket_2x09_P1.27mm_Vertical_SMD"
 			(at 189.23 74.93 0)
 			(effects
@@
 			)
 		)
-		(property "Footprint" "Capacitor_THT:C_Disc_D4.3mm_W1.9mm_P5.00mm"
+		(property "Footprint" "CollecteurDonne:Capa disc radial 5.08mm"
 			(at 178.7652 109.22 0)
 			(effects
@@
 			)
 		)
-		(property "Footprint" ""
+		(property "Footprint" "CollecteurDonne:ESP32-S3-DEVKITC-1-N8R8"
 			(at 193.04 101.6 0)
 			(effects
@@
 			)
 		)
-		(property "Footprint" "MountingHole:MountingHole_3.2mm_M3_ISO14580"
+		(property "Footprint" "CollecteurDonne:MountingHole_2.2mm_M2_ISO7380"
 			(at 248.92 29.21 0)
 			(effects
@@
 			)
 		)
-		(property "Footprint" "Capacitor_THT:C_Disc_D4.3mm_W1.9mm_P5.00mm"
+		(property "Footprint" "CollecteurDonne:Capa disc radial 5.08mm"
 			(at 163.5252 72.39 0)
 			(effects

Commit message: Update_Schematic_PCB
Parts:
- removed U6: ~, Connector_PinSocket_1.27mm:PinSocket_2x09_P1.27mm_Vertical_SMD, symbol CollecteurDonneLIB:OV2640
- added J9: Conn_02x09_Odd_Even, Connector_PinSocket_2.54mm:PinSocket_2x09_P2.54mm_Vertical, symbol Connector_Generic:Conn_02x09_Odd_Even
- C1, C7: footprint CollecteurDonne:Capa disc radial 5.08mm -> CollecteurDonne:C_Disc_D5.0mm_W2.5mm_P5.00mm
- J2: footprint CollecteurDonne:ESP32-S3-DEVKITC-1-N8R8 -> (none)
Connections:
- net +VCC_Alim: now also J9.1 (Pin_1)
- net D0: now also J9.8 (Pin_8)
- net D1: now also J9.9 (Pin_9)
- net D2: now also J9.10 (Pin_10)
- net D3: now also J9.11 (Pin_11)
- net D4: now also J9.12 (Pin_12)
- net D5: now also J9.13 (Pin_13)
- net D6: now also J9.14 (Pin_14)
- net D7: now also J9.15 (Pin_15)
- net DCLK: now also J9.16 (Pin_16)
- net GND: now also J9.2 (Pin_2)
- net HREF: now also J9.5 (Pin_5)
- net PWDN: now also J9.18 (Pin_18)
- net RST: now also J9.7 (Pin_7)
- net SCL: now also J9.4 (Pin_4)
- net SDA: now also J9.6 (Pin_6)
- net VREF: now also J9.3 (Pin_3)
Changed lines of the file:
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@@
-	)
-	(symbol
-		(lib_name "OV2640_1")
-		(lib_id "CollecteurDonneLIB:OV2640")
-		(at 189.23 74.93 0)
-		(unit 1)
-		(exclude_from_sim no)
-		(in_bom yes)
-		(on_board yes)
-		(dnp no)
-		(fields_autoplaced yes)
-		(property "Reference" "U6"
-			(at 190.5 59.69 0)
-			(effects
-				(font
-					(size 1.27 1.27)
-				)
-			)
-		)
-		(property "Value" "~"
-			(at 190.5 62.23 0)
-			(effects
-				(font
-					(size 1.27 1.27)
-				)
-			)
-		)
-		(property "Footprint" "Connector_PinSocket_1.27mm:PinSocket_2x09_P1.27mm_Vertical_SMD"
-			(at 189.23 74.93 0)
-			(effects
-				(font
-					(size 1.27 1.27)
-				)
-				(hide yes)
-			)
-		)
-		(property "Datasheet" ""
-			(at 189.23 74.93 0)
-			(effects
-				(font
-					(size 1.27 1.27)
-				)
-				(hide yes)
-			)
-		)
-		(property "Description" ""
-			(at 189.23 74.93 0)
-			(effects
-				(font
-					(size 1.27 1.27)
-				)
-				(hide yes)
-			)
-		)
-		(pin "2"
-		)
-		(pin "8"
-		)
-		(pin "9"
-		)
-		(pin "15"
-		)
-		(pin "17"
-		)
-		(pin "12"
-		)
-		(pin "7"
-		)
-		(pin "16"
-		)
-		(pin "6"
-		)
-		(pin "10"
-		)
-		(pin "3"
-		)
-		(pin "18"
-		)
-		(pin "4"
-		)
-		(pin "14"
-		)
-		(pin "5"
-		)
-		(pin "13"
-		)
-		(pin "11"
-		)
-		(pin "1"
-		)
-		(instances
-			(project ""
-				(path "/77f264da-4c84-4b0c-9d20-4392731765e6/90e676b5-e192-40ef-8f2d-7a9315f03418"
-					(reference "U6")
-					(unit 1)
-				)
-			)
-		)
 	)
 	(symbol
@@
 			)
 		)
-		(property "Footprint" "CollecteurDonne:Capa disc radial 5.08mm"
+		(property "Footprint" "CollecteurDonne:C_Disc_D5.0mm_W2.5mm_P5.00mm"
 			(at 178.7652 109.22 0)
 			(effects
@@
 			)
 		)
-		(property "Footprint" "CollecteurDonne:ESP32-S3-DEVKITC-1-N8R8"
+		(property "Footprint" ""
 			(at 193.04 101.6 0)
 			(effects
@@
 				(path "/77f264da-4c84-4b0c-9d20-4392731765e6/90e676b5-e192-40ef-8f2d-7a9315f03418"
 					(reference "J2")
+					(unit 1)
+				)
+			)
+		)
+	)
+	(symbol
+		(lib_id "Connector_Generic:Conn_02x09_Odd_Even")
+		(at 189.23 74.93 0)
+		(unit 1)
+		(exclude_from_sim no)
+		(in_bom yes)
+		(on_board yes)
+		(dnp no)
+		(fields_autoplaced yes)
+		(property "Reference" "J9"
+			(at 190.5 58.42 0)
+			(effects
+				(font
+					(size 1.27 1.27)
+				)
+			)
+		)
+		(property "Value" "Conn_02x09_Odd_Even"
+			(at 190.5 60.96 0)
+			(effects
+				(font
+					(size 1.27 1.27)
+				)
+			)
+		)
+		(property "Footprint" "Connector_PinSocket_2.54mm:PinSocket_2x09_P2.54mm_Vertical"
+			(at 189.23 74.93 0)
+			(effects
+				(font
+					(size 1.27 1.27)
+				)
+				(hide yes)
+			)
+		)
+		(property "Datasheet" "~"
+			(at 189.23 74.93 0)
+			(effects
+				(font
+					(size 1.27 1.27)
+				)
+				(hide yes)
+			)
+		)
+		(property "Description" "Generic connector, double row, 02x09, odd/even pin numbering scheme (row 1 odd numbers, row 2 even numbers), script generated (kicad-library-utils/schlib/autogen/connector/)"
+			(at 189.23 74.93 0)
+			(effects
+				(font
+					(size 1.27 1.27)
+				)
+				(hide yes)
+			)
+		)
+		(pin "3"
+		)
+		(pin "9"
+		)
+		(pin "13"
+		)
+		(pin "1"
+		)
+		(pin "5"
+		)
+		(pin "7"
+		)
+		(pin "11"
+		)
+		(pin "12"
+		)
+		(pin "18"
+		)
+		(pin "2"
+		)
+		(pin "17"
+		)
+		(pin "15"
+		)
+		(pin "4"
+		)
+		(pin "16"
+		)
+		(pin "6"
+		)
+		(pin "8"
+		)
+		(pin "10"
+		)
+		(pin "14"
+		)
+		(instances
+			(project ""
+				(path "/77f264da-4c84-4b0c-9d20-4392731765e6/90e676b5-e192-40ef-8f2d-7a9315f03418"
+					(reference "J9")
 					(unit 1)
 				)
@@
 			)
 		)
-		(property "Footprint" "CollecteurDonne:Capa disc radial 5.08mm"
+		(property "Footprint" "CollecteurDonne:C_Disc_D5.0mm_W2.5mm_P5.00mm"
 			(at 163.5252 72.39 0)
 			(effects

Commit message: Update_PCB
Parts:
- removed H5, H6: MountingHole, CollecteurDonne:MountingHole_2.2mm_M2_ISO7380, symbol Mechanical:MountingHole
- added Q4: IRF540N, Package_TO_SOT_THT:TO-220-3_Horizontal_TabDown, symbol Transistor_FET:IRF540N
- added R5: 1k, CollecteurDonne:R_Axial_DIN0207_L6.3mm_D2.5mm_P10.16mm_Horizontal, symbol Device:R_US
- J2: footprint (none) -> Connector_PinHeader_2.54mm:PinHeader_1x02_P2.54mm_Vertical
- J9: footprint Connector_PinSocket_2.54mm:PinSocket_2x09_P2.54mm_Vertical -> CollecteurDonne:OV2640
Connections:
- net GND: now also Q4.3 (S); no longer C7.2, J2.2 (Pin_2)
- new net: Q4.1 (G), R5.2
- new net: C7.2, J2.2 (Pin_2), Q4.2 (D)
- new net LED_IR: R5.1
Changed lines of the file:
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@@
 	)
 	(junction
-		(at 177.8 101.6)
+		(at 187.96 109.22)
 		(diameter 0)
 		(color 0 0 0 0)
 	)
 	(junction
-		(at 187.96 120.65)
+		(at 177.8 101.6)
 		(diameter 0)
 		(color 0 0 0 0)
@@
 	(wire
 		(pts
+			(xy 157.48 116.84) (xy 158.75 116.84)
+		)
+		(stroke
+			(width 0)
+			(type default)
+		)
+	)
+	(wire
+		(pts
 			(xy 196.85 74.93) (xy 200.66 74.93)
 		)
@@
 	(wire
 		(pts
-			(xy 177.8 109.22) (xy 177.8 120.65)
+			(xy 177.8 101.6) (xy 187.96 101.6)
 		)
 		(stroke
@@
 	(wire
 		(pts
-			(xy 177.8 101.6) (xy 187.96 101.6)
+			(xy 177.8 109.22) (xy 187.96 109.22)
 		)
 		(stroke
@@
 	(wire
 		(pts
-			(xy 177.8 120.65) (xy 187.96 120.65)
+			(xy 196.85 82.55) (xy 200.66 82.55)
 		)
 		(stroke
@@
 	(wire
 		(pts
-			(xy 196.85 82.55) (xy 200.66 82.55)
+			(xy 187.96 111.76) (xy 187.96 109.22)
+		)
+		(stroke
+			(width 0)
+			(type default)
+		)
+	)
+	(wire
+		(pts
+			(xy 187.96 121.92) (xy 187.96 123.19)
 		)
 		(stroke
@@
 	(wire
 		(pts
-			(xy 187.96 104.14) (xy 187.96 120.65)
+			(xy 187.96 104.14) (xy 187.96 109.22)
 		)
 		(stroke
@@
 	(wire
 		(pts
-			(xy 180.34 82.55) (xy 184.15 82.55)
+			(xy 166.37 116.84) (xy 180.34 116.84)
 		)
 		(stroke
@@
 	(wire
 		(pts
-			(xy 187.96 123.19) (xy 187.96 120.65)
+			(xy 180.34 82.55) (xy 184.15 82.55)
 		)
 		(stroke
@@
 		)
 	)
+	(hierarchical_label "LED_IR"
+		(shape input)
+		(at 157.48 116.84 180)
+		(effects
+			(font
+				(size 1.27 1.27)
+			)
+			(justify right)
+		)
+	)
 	(hierarchical_label "+VCC_Alim"
 		(shape input)
@@
 	)
 	(symbol
-		(lib_id "Mechanical:MountingHole")
-		(at 248.92 35.56 0)
+		(lib_id "Device:R_US")
+		(at 162.56 116.84 90)
 		(unit 1)
 		(exclude_from_sim no)
-		(in_bom no)
+		(in_bom yes)
 		(on_board yes)
 		(dnp no)
 		(fields_autoplaced yes)
-		(property "Reference" "H6"
-			(at 251.46 34.2899 0)
+		(property "Reference" "R5"
+			(at 162.56 110.49 90)
 			(effects
 				(font
 					(size 1.27 1.27)
 				)
-				(justify left)
 			)
 		)
-		(property "Value" "MountingHole"
-			(at 251.46 36.8299 0)
+		(property "Value" "1k"
+			(at 162.56 113.03 90)
 			(effects
 				(font
 					(size 1.27 1.27)
 				)
-				(justify left)
 			)
 		)
-		(property "Footprint" "CollecteurDonne:MountingHole_2.2mm_M2_ISO7380"
-			(at 248.92 35.56 0)
+		(property "Footprint" "CollecteurDonne:R_Axial_DIN0207_L6.3mm_D2.5mm_P10.16mm_Horizontal"
+			(at 162.814 115.824 90)
 			(effects
 				(font
@@
 		)
 		(property "Datasheet" "~"
-			(at 248.92 35.56 0)
-			(effects
-				(font
-					(size 1.27 1.27)
-				)
-				(hide yes)
-			)
-		)
-		(property "Description" "Mounting Hole without connection"
-			(at 248.92 35.56 0)
+			(at 162.56 116.84 0)
 			(effects
 				(font
@@
 			)
 		)
-		(property "Fabricant" ""
-			(at 248.92 35.56 0)
+		(property "Description" "Resistor, US symbol"
+			(at 162.56 116.84 0)
 			(effects
 				(font
@@
 			)
 		)
-		(property "Fournisseur" ""
-			(at 248.92 35.56 0)
-			(effects
-				(font
-					(size 1.27 1.27)
-				)
-				(hide yes)
-			)
-		)
-		(property "Ref Fabricant" ""
-			(at 248.92 35.56 0)
-			(effects
-				(font
-					(size 1.27 1.27)
-				)
-				(hide yes)
-			)
-		)
-		(property "Ref Fournisseur" ""
-			(at 248.92 35.56 0)
-			(effects
-				(font
-					(size 1.27 1.27)
-				)
-				(hide yes)
-			)
+		(pin "1"
 		)
-		(property "Sim.Type" ""
-			(at 248.92 35.56 0)
-			(effects
-				(font
-					(size 1.27 1.27)
-				)
-				(hide yes)
-			)
+		(pin "2"
 		)
 		(instances
-			(project "Main"
+			(project ""
 				(path "/77f264da-4c84-4b0c-9d20-4392731765e6/90e676b5-e192-40ef-8f2d-7a9315f03418"
-					(reference "H6")
+					(reference "R5")
 					(unit 1)
 				)
@@
 	)
 	(symbol
+		(lib_id "Transistor_FET:IRF540N")
+		(at 185.42 116.84 0)
+		(unit 1)
+		(exclude_from_sim no)
+		(in_bom yes)
+		(on_board yes)
+		(dnp no)
+		(fields_autoplaced yes)
+		(property "Reference" "Q4"
+			(at 191.77 115.5699 0)
+			(effects
+				(font
+					(size 1.27 1.27)
+				)
+				(justify left)
+			)
+		)
+		(property "Value" "IRF540N"
+			(at 191.77 118.1099 0)
+			(effects
+				(font
+					(size 1.27 1.27)
+				)
+				(justify left)
+			)
+		)
+		(property "Footprint" "Package_TO_SOT_THT:TO-220-3_Horizontal_TabDown"
+			(at 190.5 118.745 0)
+			(effects
+				(font
+					(size 1.27 1.27)
+					(italic yes)
+				)
+				(justify left)
+				(hide yes)
+			)
+		)
+		(property "Datasheet" "http://www.irf.com/product-info/datasheets/data/irf540n.pdf"
+			(at 190.5 120.65 0)
+			(effects
+				(font
+					(size 1.27 1.27)
+				)
+				(justify left)
+				(hide yes)
+			)
+		)
+		(property "Description" "33A Id, 100V Vds, HEXFET N-Channel MOSFET, TO-220"
+			(at 185.42 116.84 0)
+			(effects
+				(font
+					(size 1.27 1.27)
+				)
+				(hide yes)
+			)
+		)
+		(pin "2"
+		)
+		(pin "1"
+		)
+		(pin "3"
+		)
+		(instances
+			(project ""
+				(path "/77f264da-4c84-4b0c-9d20-4392731765e6/90e676b5-e192-40ef-8f2d-7a9315f03418"
+					(reference "Q4")
+					(unit 1)
+				)
+			)
+		)
+	)
+	(symbol
 		(lib_id "Connector_Generic:Conn_01x02")
 		(at 193.04 101.6 0)
@@
 			)
 		)
-		(property "Footprint" ""
+		(property "Footprint" "Connector_PinHeader_2.54mm:PinHeader_1x02_P2.54mm_Vertical"
 			(at 193.04 101.6 0)
 			(effects
@@
 			)
 		)
-		(property "Footprint" "Connector_PinSocket_2.54mm:PinSocket_2x09_P2.54mm_Vertical"
+		(property "Footprint" "CollecteurDonne:OV2640"
 			(at 189.23 74.93 0)
 			(effects
@@
 					(unit 1)
 				)
-			)
-		)
-	)
-	(symbol
-		(lib_id "Mechanical:MountingHole")
-		(at 248.92 29.21 0)
-		(unit 1)
-		(exclude_from_sim no)
-		(in_bom no)
-		(on_board yes)
-		(dnp no)
-		(fields_autoplaced yes)
-		(property "Reference" "H5"
-			(at 251.46 27.9399 0)
-			(effects
-				(font
-					(size 1.27 1.27)
-				)
-				(justify left)
-			)
-		)
-		(property "Value" "MountingHole"
-			(at 251.46 30.4799 0)
-			(effects
-				(font
-					(size 1.27 1.27)
-				)
-				(justify left)
-			)
-		)
-		(property "Footprint" "CollecteurDonne:MountingHole_2.2mm_M2_ISO7380"
-			(at 248.92 29.21 0)
-			(effects
-				(font
-					(size 1.27 1.27)
-				)
-				(hide yes)
-			)
-		)
-		(property "Datasheet" "~"
-			(at 248.92 29.21 0)
-			(effects
-				(font
-					(size 1.27 1.27)
-				)
-				(hide yes)
-			)
-		)
-		(property "Description" "Mounting Hole without connection"
-			(at 248.92 29.21 0)
-			(effects
-				(font
-					(size 1.27 1.27)
-				)
-				(hide yes)
-			)
-		)
-		(property "Fabricant" ""
-			(at 248.92 29.21 0)
-			(effects
-				(font
-					(size 1.27 1.27)
-				)
-				(hide yes)
-			)
-		)
-		(property "Fournisseur" ""
-			(at 248.92 29.21 0)
-			(effects
-				(font
-					(size 1.27 1.27)
-				)
-				(hide yes)
-			)
-		)
-		(property "Ref Fabricant" ""
-			(at 248.92 29.21 0)
-			(effects
-				(font
-					(size 1.27 1.27)
-				)
-				(hide yes)
-			)
-		)
-		(property "Ref Fournisseur" ""
-			(at 248.92 29.21 0)
-			(effects
-				(font
-					(size 1.27 1.27)
-				)
-				(hide yes)
-			)
-		)
-		(property "Sim.Type" ""
-			(at 248.92 29.21 0)
-			(effects
-				(font
-					(size 1.27 1.27)
-				)
-				(hide yes)
-			)
-		)
-		(instances
-			(project "Main"
-				(path "/77f264da-4c84-4b0c-9d20-4392731765e6/90e676b5-e192-40ef-8f2d-7a9315f03418"
-					(reference "H5")
-					(unit 1)
-				)
