File: Architecture/Main-REVA2/Stockage.kicad_sch (KiCad schematic)
At the start: 3 parts, among them J5 Conn_01x06

Commit message: Update_Schematic
Other:
- company: (none) -> Polytech Nantes - ETN4
- title: (none) -> Collecteur de données Animalières
- moved on the sheet: C4
Changed lines of the file:
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@@
 	(generator_version "9.0")
 	(paper "A4")
+	(title_block
+		(title "Collecteur de données Animalières")
+		(date "2025-11-28")
+		(rev "A2")
+		(company "Polytech Nantes - ETN4")
+		(comment 1 "Architecture Collectuer de données")
+		(comment 2 "Stockage Page")
+	)
 	(rectangle
 		(start 162.56 81.28)
@@
 	(wire
 		(pts
-			(xy 111.76 102.87) (xy 116.84 102.87)
+			(xy 110.49 99.06) (xy 115.57 99.06)
 		)
 		(stroke
@@
 	(wire
 		(pts
-			(xy 111.76 110.49) (xy 116.84 110.49)
+			(xy 110.49 106.68) (xy 115.57 106.68)
 		)
 		(stroke
@@
 	(hierarchical_label "VCC"
 		(shape input)
-		(at 111.76 102.87 180)
+		(at 110.49 99.06 180)
 		(effects
 			(font
@@
 	(hierarchical_label "GND"
 		(shape input)
-		(at 111.76 110.49 180)
+		(at 110.49 106.68 180)
 		(effects
 			(font
@@
 	(symbol
 		(lib_id "Device:C")
-		(at 116.84 106.68 0)
+		(at 115.57 102.87 0)
 		(unit 1)
 		(exclude_from_sim no)
@@
 		(dnp no)
 		(property "Reference" "C4"
-			(at 110.744 105.664 0)
+			(at 109.474 101.854 0)
 			(effects
 				(font
@@
 		)
 		(property "Value" "100nF"
-			(at 108.204 107.696 0)
+			(at 106.934 103.886 0)
 			(effects
 				(font
@@
 		)
 		(property "Footprint" ""
-			(at 117.8052 110.49 0)
+			(at 116.5352 106.68 0)
 			(effects
 				(font
@@
 		)
 		(property "Datasheet" "~"
-			(at 116.84 106.68 0)
+			(at 115.57 102.87 0)
 			(effects
 				(font
@@
 		)
 		(property "Description" "Unpolarized capacitor"
-			(at 116.84 106.68 0)
-			(effects
-				(font
+			(at 115.57 102.87 0)
+			(effects
+				(font

Commit message: Update
Parts:
- C4: footprint (none) -> Capacitor_THT:C_Disc_D4.3mm_W1.9mm_P5.00mm; Fabricant (none) -> KEMET; Fournisseur (none) -> RS; Ref Fabricant (none) -> C0805C104K4RACTU; Ref Fournisseur (none) -> 648-0957
- U2: value ~ -> SD_CARD; Fabricant (none) -> Sandisk; Fournisseur (none) -> RS; Ref Fabricant (none) -> SDSQUA4-032G-GN6MA; Ref Fournisseur (none) -> 283-6581
Changed lines of the file:
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@@
+			)
+		)
+		(property "Fabricant" ""
+			(at 138.43 101.6 0)
+			(effects
+				(font
+					(size 1.27 1.27)
+				)
+				(hide yes)
+			)
+		)
+		(property "Fournisseur" ""
+			(at 138.43 101.6 0)
+			(effects
+				(font
+					(size 1.27 1.27)
+				)
+				(hide yes)
+			)
+		)
+		(property "Ref Fabricant" ""
+			(at 138.43 101.6 0)
+			(effects
+				(font
+					(size 1.27 1.27)
+				)
+				(hide yes)
+			)
+		)
+		(property "Ref Fournisseur" ""
+			(at 138.43 101.6 0)
+			(effects
+				(font
+					(size 1.27 1.27)
+				)
+				(hide yes)
+			)
+		)
+		(property "Sim.Type" ""
+			(at 138.43 101.6 0)
+			(effects
+				(font
+					(size 1.27 1.27)
+				)
+				(hide yes)
 			)
 		)
@@
 			)
 		)
-		(property "Value" "~"
-			(at 175.26 104.14 0)
+		(property "Value" "SD_CARD"
+			(at 166.37 110.236 0)
 			(effects
 				(font
@@
 		)
 		(property "Description" ""
+			(at 170.18 104.14 0)
+			(effects
+				(font
+					(size 1.27 1.27)
+				)
+				(hide yes)
+			)
+		)
+		(property "Fabricant" "Sandisk"
+			(at 170.18 104.14 0)
+			(effects
+				(font
+					(size 1.27 1.27)
+				)
+				(hide yes)
+			)
+		)
+		(property "Fournisseur" "RS"
+			(at 170.18 104.14 0)
+			(effects
+				(font
+					(size 1.27 1.27)
+				)
+				(hide yes)
+			)
+		)
+		(property "Ref Fabricant" "SDSQUA4-032G-GN6MA"
+			(at 170.18 104.14 0)
+			(effects
+				(font
+					(size 1.27 1.27)
+				)
+				(hide yes)
+			)
+		)
+		(property "Ref Fournisseur" "283-6581"
+			(at 170.18 104.14 0)
+			(effects
+				(font
+					(size 1.27 1.27)
+				)
+				(hide yes)
+			)
+		)
+		(property "Sim.Type" ""
 			(at 170.18 104.14 0)
 			(effects
@@
 			)
 		)
-		(property "Footprint" ""
+		(property "Footprint" "Capacitor_THT:C_Disc_D4.3mm_W1.9mm_P5.00mm"
 			(at 116.5352 106.68 0)
 			(effects
@@
 			(at 115.57 102.87 0)
 			(effects
+				(font
+					(size 1.27 1.27)
+				)
+				(hide yes)
+			)
+		)
+		(property "Fabricant" "KEMET"
+			(at 115.57 102.87 0)
+			(effects
+				(font
+					(size 1.27 1.27)
+				)
+				(hide yes)
+			)
+		)
+		(property "Fournisseur" "RS"
+			(at 115.57 102.87 0)
+			(effects
+				(font
+					(size 1.27 1.27)
+				)
+				(hide yes)
+			)
+		)
+		(property "Ref Fabricant" "C0805C104K4RACTU"
+			(at 115.57 102.87 0)
+			(effects
+				(font
+					(size 1.27 1.27)
+				)
+				(hide yes)
+			)
+		)
+		(property "Ref Fournisseur" "648-0957"
+			(at 115.57 102.87 0)
+			(effects
+				(font
+					(size 1.27 1.27)
+				)
+				(hide yes)
+			)
+		)
+		(property "Sim.Type" ""
+			(at 115.57 102.87 0)
+			(effects

Commit message: Update_Sche
Parts:
- C4: footprint Capacitor_THT:C_Disc_D4.3mm_W1.9mm_P5.00mm -> CollecteurDonne:Capa disc radial 5.08mm
Changed lines of the file:
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@@
 		(exclude_from_sim no)
 		(in_bom yes)
-		(on_board yes)
+		(on_board no)
 		(dnp no)
 		(property "Reference" "U2"
@@
 			)
 		)
-		(property "Footprint" "Capacitor_THT:C_Disc_D4.3mm_W1.9mm_P5.00mm"
+		(property "Footprint" "CollecteurDonne:Capa disc radial 5.08mm"
 			(at 116.5352 106.68 0)
 			(effects

Commit message: Update_Schematic_PCB
Parts:
- C4: footprint CollecteurDonne:Capa disc radial 5.08mm -> CollecteurDonne:C_Disc_D5.0mm_W2.5mm_P5.00mm
Changed lines of the file:
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@@
 			)
 		)
-		(property "Footprint" "CollecteurDonne:Capa disc radial 5.08mm"
+		(property "Footprint" "CollecteurDonne:C_Disc_D5.0mm_W2.5mm_P5.00mm"
 			(at 116.5352 106.68 0)
 			(effects

Commit message: Update_PCB
Parts:
- J5: footprint (none) -> Connector_PinHeader_2.54mm:PinHeader_1x06_P2.54mm_Vertical
Changed lines of the file:
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@@
 			)
 		)
-		(property "Footprint" ""
+		(property "Footprint" "Connector_PinHeader_2.54mm:PinHeader_1x06_P2.54mm_Vertical"
 			(at 138.43 101.6 0)
 			(effects
