File: Architecture/Main-REVA2/Main.kicad_pcb (KiCad board)
At the start: 2 copper layers, 100 x 100 mm, 61 parts, among them J1 Conn_01x04, J10 IN, J11 110990030, J12 110990030, J14 OUT_5V_ALI, J16 OUT_5V_PWR, J17 Barrel_Jack_Switch_Pin3Ring, J2 Conn_01x02, J3 Conn_01x03, J4 Conn_01x04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

Commit message: Update_28_01_2025
Parts:
- moved U4 1.77 mm to (148.0, 83.3)
- moved U5 0.38 mm to (146.0, 132.0)
Connections:
- J9 pad 7: GND -> /Cam/+VCC_Alim
- U4 pad J1_10: /Transmission/TX -> /Sensors/TX0
- U4 pad J1_11: /Transmission/RX -> /Sensors/RX0
- U4 pad J1_13: /Cam/HREF -> /Cam/D1
- U4 pad J1_14: /Power/VOLTAGE_BAT -> /Cam/D0
- U4 pad J1_20: /Power/PWR_U/D -> /Cam/DCLK
- U4 pad J1_4: /Sensors/PIR_MOUV -> /Cam/D7
- U4 pad J1_5: /Sensors/DATA_DHT22 -> /Cam/D6
- U4 pad J1_6: /Sensors/ENA_GPS -> /Cam/D5
- U4 pad J1_7: /Cam/D1 -> /Cam/D4
- U4 pad J1_8: /Cam/D6 -> /Cam/D3
- U4 pad J1_9: /Cam/D7 -> /Cam/D2
- U4 pad J3_10: /Cam/D2 -> /Sensors/DATA_DHT22
- U4 pad J3_15: /Cam/D0 -> /uc/D45
- U4 pad J3_16: /Cam/DCLK -> /uc/D48
- U4 pad J3_17: /Cam/D3 -> /Power/VOLTAGE_BAT
- U4 pad J3_18: /Cam/D5 -> /Sensors/ENA_GPS
- U4 pad J3_4: /Cam/VREF -> /Sensors/PIR_MOUV
- U4 pad J3_5: /uc/D2 -> /Power/PWR_U/D
- U4 pad J3_6: /Sensors/TX0 -> /Transmission/TX
- U4 pad J3_7: /Sensors/RX0 -> /Transmission/RX
- U4 pad J3_8: /Cam/D4 -> /Cam/VREF
- U4 pad J3_9: /Cam/D2 -> /Cam/HREF
Routing:
- removed copper zone on F.Cu, net GND

Commit message: Update_PCB
Parts:
- removed H5, H6: MountingHole, CollecteurDonne:MountingHole_2.2mm_M2_ISO7380
- added Q4: IRF540N, Package_TO_SOT_THT:TO-220-3_Horizontal_TabDown, B.Cu at (154.4, 108.3)
- added R5: 1k, CollecteurDonne:R_Axial_DIN0207_L6.3mm_D2.5mm_P10.16mm_Horizontal, B.Cu at (143.3, 91.9)
- C1: moved to F.Cu
- J9: footprint Connector_PinSocket_2.54mm:PinSocket_2x09_P2.54mm_Vertical -> CollecteurDonne:OV2640
- Q1: value BS170 -> IRF540N; footprint Package_TO_SOT_THT:TO-92_Inline -> Package_TO_SOT_THT:TO-220-3_Vertical
- moved J2 36.6 mm to (138.7, 111.5), turned to 0 degrees
- moved C7 33.1 mm to (144.3, 112.7), turned to 90 degrees
- moved J9 10.0 mm to (146.3, 144.6)
- moved D1 9.88 mm to (170.2, 130.6)
- moved R19 5.79 mm to (150.4, 85.3)
- moved R18 5.79 mm to (150.4, 77.7)
- moved C2 3.52 mm to (110.2, 60.9)
- moved J12 2.21 mm to (109.2, 126.2)
- moved C16 2.21 mm to (116.8, 126.8)
- moved C17 2.21 mm to (104.1, 126.7)
- moved J11 2.21 mm to (121.9, 126.2)
- moved C19 2.13 mm to (121.9, 106.3)
- moved Q1 1.86 mm to (106.7, 61.0)
- moved J6 1.60 mm to (124.5, 64.4)
- moved C6 0.94 mm to (122.0, 139.4)
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Connections:
- C7 pad 2: GND -> Net-(J2-Pin_2)
- J2 pad 2: GND -> Net-(J2-Pin_2)
- Q1 pad 1: GND -> Net-(Q1-G)
- Q1 pad 2: Net-(Q1-G) -> GND
- U4 pad J3_16: /uc/D48 -> /Cam/LED_IR

Commit message: Update_30_01_2026
Parts:
- moved J9 24.0 mm to (146.3, 120.6), turned to -90 degrees
- moved U5 5.16 mm to (146.0, 137.2)

Commit message: update_01_02_2026
Parts:
- added JP1: Jumper_2_Bridged, Connector_PinHeader_2.54mm:PinHeader_1x02_P2.54mm_Vertical, F.Cu at (176.3, 83.8)
- C1: moved to B.Cu
- moved C1 36.0 mm to (133.6, 124.4), turned to 90 degrees
- moved D1 9.32 mm to (166.1, 122.2)
- moved U5 3.13 mm to (147.8, 134.6)
- moved R9 2.87 mm to (182.9, 84.8)
- moved C11 1.79 mm to (182.1, 109.7), turned to 90 degrees
- moved Q1 1.52 mm to (105.2, 61.0)
- moved J9 1.26 mm to (147.6, 120.6)
- moved J7 1.03 mm to (113.3, 59.2)
- moved C2 0.94 mm to (109.2, 60.9)
- moved D3 0.51 mm to (140.2, 62.5)
- moved R3 0.51 mm to (103.6, 75.9)
Connections:
- Q3 pad 3: /Cam/+VCC_Alim -> Net-(JP1-B)
- R9 pad 1: /Cam/+VCC_Alim -> Net-(JP1-B)
Routing:
- net GND: track 0.00 -> 507.1 mm
- net +5V: track 0.00 -> 279.5 mm, vias 0 -> 1
- net /Cam/+VCC_Alim: track 0.00 -> 174.8 mm
- net /Cam/SDA: track 0.00 -> 106.0 mm, vias 0 -> 1
- net /Power/VOLTAGE_BAT: track 0.00 -> 105.4 mm, vias 0 -> 1
- net /Cam/SCL: track 0.00 -> 104.7 mm, vias 0 -> 1
- net +12V: track 0.00 -> 94.3 mm, vias 0 -> 1
- net /Cam/PWDN: track 0.00 -> 81.9 mm
- net /Power/PWR_U/D: track 0.00 -> 81.1 mm, vias 0 -> 1
- net /Sensors/TX0: track 0.00 -> 71.9 mm, vias 0 -> 1
- net /Sensors/RX0: track 0.00 -> 60.3 mm, vias 0 -> 1
- net /Cam/DCLK: track 0.00 -> 59.9 mm
- net /Cam/D1: track 0.00 -> 45.1 mm
- net /Cam/D0: track 0.00 -> 44.9 mm
- net /Sensors/PIR_MOUV: track 0.00 -> 44.8 mm
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- added copper zone on F.Cu, net GND
Other:
- board text added: "AMP"

Commit message: Update_6_02_2026
Parts:
- added C18: 100uF, CollecteurDonne:C_Radial_D10.0mm_H16.0mm_P5.00mm, B.Cu at (145.8, 65.0)
- added R6: 10k, CollecteurDonne:R_Axial_DIN0207_L6.3mm_D2.5mm_P10.16mm_Horizontal, F.Cu at (114.0, 139.2)
- C12: value 100µF -> 470µF
- moved U5 234.8 mm to (-28.4, -20.6)
- moved D3 12.3 mm to (147.8, 72.1), turned to 180 degrees
- moved C20 5.66 mm to (154.9, 65.0), turned to 90 degrees
- moved C6 1.13 mm to (123.2, 139.2)
- moved D2 1.11 mm to (187.5, 136.7)
- moved C17 0.54 mm to (104.1, 127.3)
- moved C16 0.50 mm to (116.8, 127.3)
- moved J17 0.39 mm to (177.9, 134.0)
- moved C3 0.33 mm to (121.9, 87.3)
Routing:
- net GND: track 507.1 -> 62.9 mm
- net +5V: track 279.5 -> 31.2 mm, vias 1 -> 0
- net /Cam/+VCC_Alim: track 174.8 -> 0.00 mm
- net /Cam/SDA: track 106.0 -> 0.00 mm, vias 1 -> 0
- net /Power/VOLTAGE_BAT: track 105.4 -> 0.00 mm, vias 1 -> 0
- net /Cam/SCL: track 104.7 -> 0.00 mm, vias 1 -> 0
- net /Cam/PWDN: track 81.9 -> 0.00 mm
- net /Power/PWR_U/D: track 81.1 -> 0.00 mm, vias 1 -> 0
- net +12V: track 94.3 -> 15.6 mm, vias 1 -> 0
- net /Sensors/TX0: track 71.9 -> 0.00 mm, vias 1 -> 0
- net /Sensors/RX0: track 60.3 -> 0.00 mm, vias 1 -> 0
- net /Cam/DCLK: track 59.9 -> 0.00 mm
- net /Cam/D1: track 45.1 -> 0.00 mm
- net /Cam/D0: track 44.9 -> 0.00 mm
- net /Transmission/RX: track 34.7 -> 0.00 mm
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
Commit message: Update_10_02_2026
Parts:
- moved U5 236.4 mm to (148.1, 136.7)
- moved C13 3.59 mm to (188.0, 101.6)
- moved C11 3.30 mm to (183.4, 106.6)
- moved J14 2.72 mm to (194.0, 94.7), turned to 0 degrees
- moved R1 1.60 mm to (195.6, 124.1)
- moved R2 1.60 mm to (185.4, 130.5)
- moved R8 1.20 mm to (175.0, 65.8)
- moved J2 1.02 mm to (139.7, 111.5)
- moved L1 0.61 mm to (179.3, 116.3)
- moved R11 0.43 mm to (191.0, 64.4)
- moved J6 0.18 mm to (124.5, 64.3)
- moved R10 0.18 mm to (179.8, 65.7)
- moved C15 0.08 mm to (195.3, 64.4)
Routing:
- net GND: track 62.9 -> 528.3 mm
- net +5V: track 31.2 -> 280.7 mm
- net /Cam/+VCC_Alim: track 0.00 -> 170.5 mm, vias 0 -> 3
- net /Cam/SDA: track 0.00 -> 122.2 mm, vias 0 -> 1
- net +12V: track 15.6 -> 128.6 mm, vias 0 -> 1
- net /Cam/SCL: track 0.00 -> 109.8 mm, vias 0 -> 2
- net /Power/VOLTAGE_BAT: track 0.00 -> 99.4 mm
- net /Power/PWR_U/D: track 0.00 -> 83.4 mm, vias 0 -> 1
- net /Cam/PWDN: track 0.00 -> 80.5 mm
- net /Transmission/TX: track 0.00 -> 67.3 mm, vias 0 -> 1
- net /Transmission/RX: track 0.00 -> 63.0 mm, vias 0 -> 2
- net /Sensors/TX0: track 0.00 -> 62.8 mm, vias 0 -> 2
- net /Sensors/RX0: track 0.00 -> 62.7 mm, vias 0 -> 2
- net /Cam/DCLK: track 0.00 -> 59.2 mm
- net /Sensors/PIR_MOUV: track 14.0 -> 65.3 mm
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- added copper zone on B.Cu, net (none)
- added copper zone on F.Cu, net (none)
- removed copper zone on B.Cu, net GND
- removed copper zone on F.Cu, net GND
Other:
- board text added: "A"
- board text added: "Collecteur de données animalières REVA2"
- board text removed: "AMP"

Commit message: Update
Parts:
- added D4: LED, LED_THT:LED_D5.0mm, F.Cu at (105.4, 90.2)
- added Q5: PN2222A, Package_TO_SOT_THT:TO-92_Inline, F.Cu at (105.4, 97.8)
- added R12: 10k, CollecteurDonne:R_Axial_DIN0207_L6.3mm_D2.5mm_P10.16mm_Horizontal, F.Cu at (104.1, 81.3)
- added R13: 1k, CollecteurDonne:R_Axial_DIN0207_L6.3mm_D2.5mm_P10.16mm_Horizontal, F.Cu at (130.0, 81.3)
Connections:
- U4 pad J3_15: /uc/D45 -> /Sensors/DEBUG
Routing:
- net +5V: track 280.7 -> 306.1 mm
- net Net-(Q5-B): track 0.00 -> 23.1 mm
- net GND: track 528.3 -> 545.1 mm
- net Net-(D4-A): track 0.00 -> 11.5 mm
- net /Sensors/DEBUG: track 0.00 -> 5.49 mm
- net Net-(D4-K): track 0.00 -> 5.08 mm
- net /Cam/+VCC_Alim: track 170.5 -> 173.8 mm
- net /Transmission/TX: track 67.3 -> 70.0 mm, vias 1 -> 2
- net /Sensors/ENA_GPS: track 35.3 -> 32.7 mm
- net /Sensors/PIR_MOUV: track 65.3 -> 62.7 mm
- net /Power/VOLTAGE_BAT: track 99.4 -> 102.0 mm
- net /Cam/HREF: track 32.5 -> 35.1 mm
- net /Cam/VREF: track 29.7 -> 32.2 mm
- net /Cam/LED_IR: track 19.5 -> 22.1 mm, vias 0 -> 1
- net /Transmission/RX: track 63.0 -> 65.1 mm
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Other:
- board text added: "DEB"
