File: Architecture/Main-REVA2/Main.kicad_sch (KiCad schematic)
At the start: 0 parts

Commit message: Update_Schematic
Parts:
- added H1, H2, H3, H4: MountingHole, symbol Mechanical:MountingHole
Connections:
- no-connect marks 5 -> 4
Other:
- sheet Cam ports: added +VCC; removed +3.3V
- sheet Power ports: added +5V_ALIM, +5V_POWER_UP; removed +3.3V_BATT, +3.3V_POWER_UP, 12V_POWER_UP, PIR_MOUV, RECHARGE_INFO
- sheet Sensors ports: added +VCC, ENA_GPS; removed +3.3V, +3.3V_BATTERY, Voltage_Batt, Voltage_Batt_value
- sheet Transmission ports: added +VCC; removed +3.3V

Commit message: Update
Parts:
- H1, H2, H3, H4: footprint (none) -> MountingHole:MountingHole_3.2mm_M3_ISO14580
Other:
- sheet Cam ports: added +VCC_Alim; removed +VCC
- sheet Power ports: added POWER_UP; removed none

Commit message: Update_Sche
Parts:
- H1, H2, H3, H4: footprint MountingHole:MountingHole_3.2mm_M3_ISO14580 -> CollecteurDonne:MountingHole_2.2mm_M2_ISO7380
Changed lines of the file:
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@@
 			)
 		)
-		(property "Footprint" "MountingHole:MountingHole_3.2mm_M3_ISO14580"
+		(property "Footprint" "CollecteurDonne:MountingHole_2.2mm_M2_ISO7380"
 			(at 90.17 185.42 0)
 			(effects
@@
 			)
 		)
-		(property "Footprint" "MountingHole:MountingHole_3.2mm_M3_ISO14580"
+		(property "Footprint" "CollecteurDonne:MountingHole_2.2mm_M2_ISO7380"
 			(at 90.17 179.07 0)
 			(effects
@@
 			)
 		)
-		(property "Footprint" "MountingHole:MountingHole_3.2mm_M3_ISO14580"
+		(property "Footprint" "CollecteurDonne:MountingHole_2.2mm_M2_ISO7380"
 			(at 111.76 179.07 0)
 			(effects
@@
 			)
 		)
-		(property "Footprint" "MountingHole:MountingHole_3.2mm_M3_ISO14580"
+		(property "Footprint" "CollecteurDonne:MountingHole_2.2mm_M2_ISO7380"
 			(at 111.76 185.42 0)
 			(effects

Commit message: Update_Schematic_PCB
Parts:
- added U5: ~, CollecteurDonne:Logo_20_20, symbol CollecteurDonneLIB:Logo
Connections:
- no-connect marks 4 -> 1
Other:
- sheet Power ports: added V_Battery; removed none
- sheet Sensors ports: added none; removed BRIGHTNESS_SENSOR
- sheet uc ports: added D16; removed D18
- note added: "Logo"
- note added: "Mechanic"
- moved on the sheet: H1, H2, H3, H4

Commit message: Update_28_01_2025
Connections:
- no-connect marks 1 -> 3
Other:
- sheet uc ports: added D38; removed none

Commit message: Update_PCB
Connections:
- no-connect marks 3 -> 2
Other:
- sheet Cam ports: added LED_IR; removed none
Changed lines of the file:
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@@
-	)
-	(no_connect
-		(at 167.64 20.32)
 	)
 	(no_connect
@@
 	)
 	(no_connect
-		(at 170.18 20.32)
+		(at 160.02 20.32)
 	)
 	(wire
@@
 	(wire
 		(pts
-			(xy 170.18 20.32) (xy 170.18 22.86)
+			(xy 160.02 20.32) (xy 160.02 22.86)
 		)
 		(stroke
@@
 	(wire
 		(pts
-			(xy 167.64 20.32) (xy 167.64 22.86)
-		)
-		(stroke
-			(width 0)
-			(type default)
-		)
-	)
-	(wire
-		(pts
 			(xy 214.63 83.82) (xy 214.63 133.35)
 		)
@@
 		(pts
 			(xy 189.23 31.75) (xy 229.87 31.75)
+		)
+		(stroke
+			(width 0)
+			(type default)
+		)
+	)
+	(wire
+		(pts
+			(xy 177.8 46.99) (xy 229.87 46.99)
 		)
 		(stroke
@@
 		)
 		(pin "D48" input
-			(at 167.64 22.86 90)
+			(at 177.8 46.99 0)
 			(effects
 				(font
@@
 		)
 		(pin "D45" input
-			(at 170.18 22.86 90)
+			(at 160.02 22.86 90)
 			(effects
 				(font
@@
 			(effects
 				(font
+					(size 1.27 1.27)
+				)
+				(justify left)
+			)
+		)
+		(pin "LED_IR" input
+			(at 229.87 46.99 180)
+			(effects
+				(font

Commit message: Update
Connections:
- no-connect marks 2 -> 1
Other:
- sheet Sensors ports: added DEBUG; removed none
Changed lines of the file:
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@@
 		(at 153.67 20.32)
 	)
-	(no_connect
-		(at 160.02 20.32)
-	)
 	(wire
 		(pts
@@
 	(wire
 		(pts
+			(xy 69.85 38.1) (xy 130.81 38.1)
+		)
+		(stroke
+			(width 0)
+			(type default)
+		)
+	)
+	(wire
+		(pts
 			(xy 161.29 107.95) (xy 161.29 115.57)
-		)
-		(stroke
-			(width 0)
-			(type default)
-		)
-	)
-	(wire
-		(pts
-			(xy 160.02 20.32) (xy 160.02 22.86)
 		)
 		(stroke
@@
 			)
 		)
+		(pin "DEBUG" input
+			(at 69.85 38.1 0)
+			(effects
+				(font
+					(size 1.27 1.27)
+				)
+				(justify right)
+			)
+		)
 		(instances
 			(project "Main"
@@
 		)
 		(pin "D45" input
-			(at 160.02 22.86 90)
-			(effects
-				(font
-					(size 1.27 1.27)
-				)
-				(justify right)
-			)
-		)
+			(at 130.81 38.1 180)
+			(effects
+				(font
+					(size 1.27 1.27)
+				)
+				(justify left)
+			)
+		)
