File: Architecture/Main-REVA2/Power.kicad_sch (KiCad schematic)
At the start: 39 parts, among them J7 1.8 - 5.5 - Battery, J8 12V - Secteur, U1 MIC4690

Commit message: Update_Schematic
Parts:
- removed C6: 22u, symbol Device:C_Polarized
- removed C7, C? (x5): 220u, symbol Device:C_Polarized
- removed C? (x2): 100nF, symbol Device:C
- removed D1, D?: D, symbol Device:D
- removed D? (x2): 1N4001, Diode_THT:D_DO-41_SOD81_P10.16mm_Horizontal, symbol Diode:1N4001
- removed D? (x3): PMEG2010AEH, Diode_SMD:D_SOD-123F, symbol Diode:PMEG2010AEH
- removed J7: 1.8 - 5.5 - Battery, symbol Connector:Screw_Terminal_01x02
- removed J8: 12V - Secteur, symbol Connector:Screw_Terminal_01x02
- removed L? (x2): 68u, symbol Device:L
- removed Q?: PMOS, symbol Simulation_SPICE:PMOS
- removed Q? (x2): PN2222A, Package_TO_SOT_THT:TO-92_Inline, symbol Transistor_BJT:PN2222A
- removed R? (x2): 1k, symbol Device:R_US
- removed R? (x3): 10k, symbol Device:R_US
- removed R? (x3): R_US, symbol Device:R_US
- removed R? (x2): 100k, symbol Device:R_US
- removed U1: MIC4690, Package_SO:SOIC-8_3.9x4.9mm_P1.27mm, symbol Regulator_Switching:MIC4690
- removed U?: TPS63000, Package_SON:Texas_DRC0010J_ThermalVias, symbol Regulator_Switching:TPS63000
- removed U?: MCP1662-xOT, Package_TO_SOT_SMD:SOT-23-5, symbol Driver_LED:MCP1662-xOT
- added C10: 1µF, symbol Device:C_Polarized
- added C11, C13, C15, C9: 100nF, symbol Device:C
- added C12, C14, C8: 100µF, symbol Device:C_Polarized
- added J10: IN, symbol Connector:Screw_Terminal_01x02
- added J9: Jack-DC, symbol Connector:Jack-DC
- added Q2: PN2222A, Package_TO_SOT_THT:TO-92_Inline, symbol Transistor_BJT:PN2222A
- added Q3: IRF9540N, Package_TO_SOT_THT:TO-220-3_Vertical, symbol Transistor_FET:IRF9540N
- added R10, R11, R7: 10k, symbol Device:R_US
- added R4: 52.3k, symbol Device:R_US
- added R8: 1k, symbol Device:R_US
- added R9: 100k, symbol Device:R_US
- added U3: MCP16311x-xMS, Package_SO:MSOP-8_3x3mm_P0.65mm, symbol Regulator_Switching:MCP16311x-xMS
- L1: value 68u -> 22µH
- R1: value 3.01k -> 100k
- R2: value 1.78k -> 25k
Connections:
- net GND: now also C10.2, C12.2, C13.2, C14.2, C15.2, C8.2, C9.2, J10.1 (Pin_1), J9.2, Q2.1 (E), R11.2, R7.2, U3.5 (GND), U3.8 (GND)
- net PWR_U/D: now also R8.1
- net VOLTAGE_BAT: now also R1.2, R2.1
- net at L1.1: now also U3.6 (SW)
- net +5V_ALIM: now reaches L1.2
- net +5V_ALIM: now also C11.2, C12.1, C13.1, Q3.3 (S), R4.1, R9.1; no longer R1.1
- new net: C10.1, U3.2 (V_{CC})
- new net: Q3.1 (G), R10.1, R9.2
- new net: R4.2, R7.1, U3.1 (Vfb)
- new net: C11.1, U3.7 (BOOST)
- new net: Q2.3 (C), R10.2
- new net: Q2.2 (B), R8.2
- new net +5V_POWER_UP: C14.1, C15.1, Q3.2 (D), R11.1
- new net V_Battery: C8.1, C9.1, J10.2 (Pin_2), J9.1, R1.1, U3.3 (EN), U3.4 (V_{IN})
Other:
- note added: "Mesure Battery Voltage"
- company: (none) -> Polytech Nantes - ETN4
- title: (none) -> Collecteur de données Animalières

Commit message: Update
Parts:
- removed J9: Jack-DC, symbol Connector:Jack-DC
- added J14, J16: IN, symbol Connector:Screw_Terminal_01x02
- added J17: Barrel_Jack_Switch_Pin3Ring, symbol Connector:Barrel_Jack_Switch_Pin3Ring
- C10: footprint (none) -> Capacitor_THT:CP_Radial_D8.0mm_P5.00mm; Fabricant (none) -> KEMET; Fournisseur (none) -> RS; Ref Fabricant (none) -> C0603C105K4PACTU; Ref Fournisseur (none) -> 691-1142
- C11, C13, C15, C9: footprint (none) -> Capacitor_THT:C_Disc_D4.3mm_W1.9mm_P5.00mm; Fabricant (none) -> KEMET; Fournisseur (none) -> RS; Ref Fabricant (none) -> C0805C104K4RACTU; Ref Fournisseur (none) -> 648-0957
- C12: footprint (none) -> Capacitor_THT:C_Disc_D4.3mm_W1.9mm_P5.00mm; Fabricant (none) -> Vishay; Fournisseur (none) -> RS; Ref Fabricant (none) -> MAL215373101E3; Ref Fournisseur (none) -> 280-6780P
- C14, C8: footprint (none) -> Capacitor_THT:CP_Radial_D8.0mm_P5.00mm; Fabricant (none) -> Vishay; Fournisseur (none) -> RS; Ref Fabricant (none) -> MAL215373101E3; Ref Fournisseur (none) -> 280-6780P
- J10: Fabricant (none) -> Amphenol; Fournisseur (none) -> RS; Ref Fabricant (none) -> OQ0232510000G; Ref Fournisseur (none) -> 446-488
- L1: Fabricant (none) -> B82462G4223M000; Fournisseur (none) -> RS; Ref Fabricant (none) -> EPCOS; Ref Fournisseur (none) -> 495-8155P
- Q2: Fabricant (none) -> ONSEMI; Fournisseur (none) -> RS; Ref Fabricant (none) -> PN2222ATA; Ref Fournisseur (none) -> 739-0381
- Q3: Fabricant (none) -> Infineon; Fournisseur (none) -> RS; Ref Fabricant (none) -> IRF9540NPBF; Ref Fournisseur (none) -> 541-1225
- R1, R9: Fabricant (none) -> Panasonic; Fournisseur (none) -> RS; Ref Fabricant (none) -> ERA6VEB1003V; Ref Fournisseur (none) -> 241-3345
- U3: Fabricant (none) -> Microchip; Fournisseur (none) -> RS; Ref Fabricant (none) -> MCP16311/2; Ref Fournisseur (none) -> 644-286
Connections:
- net +5V_ALIM: now also J14.1 (Pin_1)
- net +5V_POWER_UP: now also J16.1 (Pin_1)
- net GND: now also J14.2 (Pin_2), J16.2 (Pin_2), J17.2, J17.3
- net V_Battery: now also J17.1
- net POWER_UP: now reaches Q3.1 (G), R10.1, R9.2

Commit message: Update_Sche
Parts:
- added D1: D, CollecteurDonne:BarrelJack_Horizontal, symbol Device:D
- added D2: D, symbol Device:D
- C10, C14, C8: footprint Capacitor_THT:CP_Radial_D8.0mm_P5.00mm -> CollecteurDonne:C_polar_D5mm
- C11, C13, C15, C9: footprint Capacitor_THT:C_Disc_D4.3mm_W1.9mm_P5.00mm -> CollecteurDonne:Capa disc radial 5.08mm
- C12: footprint Capacitor_THT:C_Disc_D4.3mm_W1.9mm_P5.00mm -> CollecteurDonne:C_polar_D5mm
- J14: value IN -> OUT_5V_ALI
- J16: value IN -> OUT_5V_PWR
- J17: footprint (none) -> CollecteurDonne:BarrelJack_Horizontal
- L1, R1, R10, R11, R2, R4, R7, R8, R9: footprint (none) -> CollecteurDonne:Résistance L10mm
Connections:
- net V_Battery: now also D1.1 (K), D2.1 (K); no longer J10.2 (Pin_2), J17.1
- new net: D2.2 (A), J10.2 (Pin_2)
- new net: D1.2 (A), J17.1
Other:
- moved on the sheet: J10, J17

Commit message: Update_Schematic_PCB
Parts:
- C10, C12, C14, C8: footprint CollecteurDonne:C_polar_D5mm -> CollecteurDonne:C_Radial_D10.0mm_H16.0mm_P5.00mm
- C11, C13, C15, C9: footprint CollecteurDonne:Capa disc radial 5.08mm -> CollecteurDonne:C_Disc_D5.0mm_W2.5mm_P5.00mm
- D1: footprint CollecteurDonne:BarrelJack_Horizontal -> CollecteurDonne:D_DO-35_SOD27_P7.62mm_Horizontal
- D2: footprint (none) -> CollecteurDonne:D_DO-35_SOD27_P7.62mm_Horizontal
- J10: now not fitted
- L1, R1, R10, R11, R2, R4, R7, R8, R9: footprint CollecteurDonne:Résistance L10mm -> CollecteurDonne:R_Axial_DIN0207_L6.3mm_D2.5mm_P10.16mm_Horizontal
Changed lines of the file:
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@@
 	(wire
 		(pts
-			(xy 196.85 59.69) (xy 193.04 59.69)
-		)
-		(stroke
-			(width 0)
-			(type default)
-		)
-	)
-	(wire
-		(pts
 			(xy 95.25 49.53) (xy 95.25 52.07)
 		)
@@
 	(wire
 		(pts
-			(xy 64.77 67.31) (xy 57.15 67.31)
+			(xy 64.77 67.31) (xy 54.61 67.31)
 		)
 		(stroke
@@
 	(wire
 		(pts
-			(xy 196.85 63.5) (xy 196.85 59.69)
+			(xy 193.04 63.5) (xy 193.04 59.69)
 		)
 		(stroke
@@
 	(wire
 		(pts
-			(xy 57.15 69.85) (xy 62.23 69.85)
+			(xy 54.61 69.85) (xy 62.23 69.85)
 		)
 		(stroke
@@
 	(wire
 		(pts
+			(xy 69.85 36.83) (xy 73.66 36.83)
+		)
+		(stroke
+			(width 0)
+			(type default)
+		)
+	)
+	(wire
+		(pts
 			(xy 64.77 49.53) (xy 69.85 49.53)
 		)
@@
 		)
 	)
+	(wire
+		(pts
+			(xy 69.85 36.83) (xy 69.85 49.53)
+		)
+		(stroke
+			(width 0)
+			(type default)
+		)
+	)
 	(image
 		(at 208.28 124.46)
@@
 		)
 	)
+	(hierarchical_label "V_Battery"
+		(shape input)
+		(at 73.66 36.83 0)
+		(effects
+			(font
+				(size 1.27 1.27)
+			)
+			(justify left)
+		)
+	)
 	(hierarchical_label "+5V_ALIM"
 		(shape input)
@@
 	(hierarchical_label "POWER_UP"
 		(shape input)
-		(at 196.85 63.5 270)
+		(at 193.04 63.5 270)
 		(effects
 			(font
@@
 			)
 		)
-		(property "Footprint" "CollecteurDonne:Résistance L10mm"
+		(property "Footprint" "CollecteurDonne:R_Axial_DIN0207_L6.3mm_D2.5mm_P10.16mm_Horizontal"
 			(at 72.136 119.634 90)
 			(effects
@@
 			)
 		)
-		(property "Footprint" "CollecteurDonne:C_polar_D5mm"
+		(property "Footprint" "CollecteurDonne:C_Radial_D10.0mm_H16.0mm_P5.00mm"
 			(at 153.3652 63.5 0)
 			(effects
@@
 			)
 		)
-		(property "Footprint" "CollecteurDonne:C_polar_D5mm"
+		(property "Footprint" "CollecteurDonne:C_Radial_D10.0mm_H16.0mm_P5.00mm"
 			(at 70.8152 67.31 0)
 			(effects
@@
 			)
 		)
-		(property "Footprint" "CollecteurDonne:C_polar_D5mm"
+		(property "Footprint" "CollecteurDonne:C_Radial_D10.0mm_H16.0mm_P5.00mm"
 			(at 96.2152 67.31 0)
 			(effects
@@
 			)
 		)
-		(property "Footprint" ""
+		(property "Footprint" "CollecteurDonne:D_DO-35_SOD27_P7.62mm_Horizontal"
 			(at 64.77 57.15 0)
 			(effects
@@
 			)
 		)
-		(property "Footprint" "CollecteurDonne:Résistance L10mm"
+		(property "Footprint" "CollecteurDonne:R_Axial_DIN0207_L6.3mm_D2.5mm_P10.16mm_Horizontal"
 			(at 180.086 54.864 90)
 			(effects
@@
 			)
 		)
-		(property "Footprint" "CollecteurDonne:Résistance L10mm"
+		(property "Footprint" "CollecteurDonne:R_Axial_DIN0207_L6.3mm_D2.5mm_P10.16mm_Horizontal"
 			(at 140.716 65.024 90)
 			(effects
@@
 			)
 		)
-		(property "Footprint" "CollecteurDonne:Capa disc radial 5.08mm"
+		(property "Footprint" "CollecteurDonne:C_Disc_D5.0mm_W2.5mm_P5.00mm"
 			(at 83.5152 67.31 0)
 			(effects
@@
 			)
 		)
-		(property "Footprint" "CollecteurDonne:C_polar_D5mm"
+		(property "Footprint" "CollecteurDonne:C_Radial_D10.0mm_H16.0mm_P5.00mm"
 			(at 205.4352 63.5 0)
 			(effects
@@
 	(symbol
 		(lib_id "Connector:Screw_Terminal_01x02")
-		(at 52.07 69.85 180)
+		(at 49.53 69.85 180)
 		(unit 1)
 		(exclude_from_sim no)
 		(in_bom yes)
 		(on_board yes)
-		(dnp no)
+		(dnp yes)
 		(fields_autoplaced yes)
 		(property "Reference" "J10"
-			(at 52.07 60.96 0)
+			(at 49.53 60.96 0)
 			(effects
 				(font
@@
 		)
 		(property "Value" "IN"
-			(at 52.07 63.5 0)
+			(at 49.53 63.5 0)
 			(effects
 				(font
@@
 		)
 		(property "Footprint" ""
-			(at 52.07 69.85 0)
+			(at 49.53 69.85 0)
 			(effects
 				(font
@@
 		)
 		(property "Datasheet" "~"
-			(at 52.07 69.85 0)
+			(at 49.53 69.85 0)
 			(effects
 				(font
@@
 		)
 		(property "Description" "Generic screw terminal, single row, 01x02, script generated (kicad-library-utils/schlib/autogen/connector/)"
-			(at 52.07 69.85 0)
+			(at 49.53 69.85 0)
 			(effects
 				(font
@@
 		)
 		(property "Fabricant" "Amphenol"
-			(at 52.07 69.85 0)
+			(at 49.53 69.85 0)
 			(effects
 				(font
@@
 		)
 		(property "Fournisseur" "RS"
-			(at 52.07 69.85 0)
+			(at 49.53 69.85 0)
 			(effects
 				(font
@@
 		)
 		(property "Ref Fabricant" "OQ0232510000G"
-			(at 52.07 69.85 0)
+			(at 49.53 69.85 0)
 			(effects
 				(font
@@
 		)
 		(property "Ref Fournisseur" "446-488"
-			(at 52.07 69.85 0)
+			(at 49.53 69.85 0)
 			(effects
 				(font
@@
 		)
 		(property "Sim.Type" ""
-			(at 52.07 69.85 0)
+			(at 49.53 69.85 0)
 			(effects
 				(font
@@
 			)
 		)
-		(property "Footprint" "CollecteurDonne:Résistance L10mm"
+		(property "Footprint" "CollecteurDonne:R_Axial_DIN0207_L6.3mm_D2.5mm_P10.16mm_Horizontal"
 			(at 180.086 65.024 90)
 			(effects
@@
 			)
 		)
-		(property "Footprint" "CollecteurDonne:Résistance L10mm"
+		(property "Footprint" "CollecteurDonne:R_Axial_DIN0207_L6.3mm_D2.5mm_P10.16mm_Horizontal"
 			(at 165.354 75.184 90)
 			(effects
@@
 			)
 		)
-		(property "Footprint" "CollecteurDonne:BarrelJack_Horizontal"
+		(property "Footprint" "CollecteurDonne:D_DO-35_SOD27_P7.62mm_Horizontal"
 			(at 59.69 49.53 0)
 			(effects
@@
 			)
 		)
-		(property "Footprint" "CollecteurDonne:Capa disc radial 5.08mm"
+		(property "Footprint" "CollecteurDonne:C_Disc_D5.0mm_W2.5mm_P5.00mm"
 			(at 219.4052 63.5 0)
 			(effects
@@
 			)
 		)
-		(property "Footprint" "CollecteurDonne:Capa disc radial 5.08mm"
+		(property "Footprint" "CollecteurDonne:C_Disc_D5.0mm_W2.5mm_P5.00mm"
 			(at 166.0652 63.5 0)
 			(effects
@@
 			)
 		)
-		(property "Footprint" "CollecteurDonne:Résistance L10mm"
+		(property "Footprint" "CollecteurDonne:R_Axial_DIN0207_L6.3mm_D2.5mm_P10.16mm_Horizontal"
 			(at 233.426 59.944 90)
 			(effects
@@
 			)
 		)
-		(property "Footprint" "CollecteurDonne:Résistance L10mm"
+		(property "Footprint" "CollecteurDonne:R_Axial_DIN0207_L6.3mm_D2.5mm_P10.16mm_Horizontal"
 			(at 72.136 129.794 90)
 			(effects
@@
 			)
 		)
-		(property "Footprint" "CollecteurDonne:Capa disc radial 5.08mm"
+		(property "Footprint" "CollecteurDonne:C_Disc_D5.0mm_W2.5mm_P5.00mm"
 			(at 133.35 44.7548 0)
 			(effects
@@
 			)
 		)
-		(property "Footprint" "CollecteurDonne:Résistance L10mm"
+		(property "Footprint" "CollecteurDonne:R_Axial_DIN0207_L6.3mm_D2.5mm_P10.16mm_Horizontal"
 			(at 140.716 54.864 90)
 			(effects
@@
 			)
 		)
-		(property "Footprint" "CollecteurDonne:Résistance L10mm"
+		(property "Footprint" "CollecteurDonne:R_Axial_DIN0207_L6.3mm_D2.5mm_P10.16mm_Horizontal"
 			(at 129.54 52.07 0)
 			(effects

Commit message: Update_PCB
Parts:
- J10, J14, J16: footprint (none) -> Connector_PinHeader_2.54mm:PinHeader_1x02_P2.54mm_Vertical
Changed lines of the file:
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@@
 	(wire
 		(pts
-			(xy 95.25 46.99) (xy 95.25 49.53)
-		)
-		(stroke
-			(width 0)
-			(type default)
-		)
-	)
-	(wire
-		(pts
 			(xy 139.7 69.85) (xy 152.4 69.85)
 		)
@@
 			)
 		)
-		(property "Footprint" ""
+		(property "Footprint" "Connector_PinHeader_2.54mm:PinHeader_1x02_P2.54mm_Vertical"
 			(at 252.73 25.4 0)
 			(effects
@@
 			)
 		)
-		(property "Footprint" ""
+		(property "Footprint" "Connector_PinHeader_2.54mm:PinHeader_1x02_P2.54mm_Vertical"
 			(at 200.66 24.13 0)
 			(effects
@@
 			)
 		)
-		(property "Footprint" ""
+		(property "Footprint" "Connector_PinHeader_2.54mm:PinHeader_1x02_P2.54mm_Vertical"
 			(at 49.53 69.85 0)
 			(effects
@@
 					(unit 1)
 				)
-			)
-		)
-	)
-	(symbol
-		(lib_id "power:PWR_FLAG")
-		(at 95.25 46.99 0)
-		(unit 1)
-		(exclude_from_sim no)
-		(in_bom yes)
-		(on_board yes)
-		(dnp no)
-		(fields_autoplaced yes)
-		(property "Reference" "#FLG04"
-			(at 95.25 45.085 0)
-			(effects
-				(font
-					(size 1.27 1.27)
-				)
-				(hide yes)
-			)
-		)
-		(property "Value" "PWR_FLAG"
-			(at 95.25 41.91 0)
-			(effects
-				(font
-					(size 1.27 1.27)
-				)
-			)
-		)
-		(property "Footprint" ""
-			(at 95.25 46.99 0)
-			(effects
-				(font
-					(size 1.27 1.27)
-				)
-				(hide yes)
-			)
-		)
-		(property "Datasheet" "~"
-			(at 95.25 46.99 0)
-			(effects
-				(font
-					(size 1.27 1.27)
-				)
-				(hide yes)
-			)
-		)
-		(property "Description" "Special symbol for telling ERC where power comes from"
-			(at 95.25 46.99 0)
-			(effects
-				(font
-					(size 1.27 1.27)
-				)
-				(hide yes)
-			)
-		)
-		(pin "1"
-		)
-		(instances
-			(project ""
-				(path "/77f264da-4c84-4b0c-9d20-4392731765e6/8078826c-4446-4e50-a209-45fcf7cbe7e4"
-					(reference "#FLG04")
-					(unit 1)
-				)

Commit message: update_01_02_2026
Parts:
- added JP1: Jumper_2_Bridged, Connector_PinHeader_2.54mm:PinHeader_1x02_P2.54mm_Vertical, symbol Jumper:Jumper_2_Bridged
Connections:
- net +5V_ALIM: now also JP1.1 (A); no longer Q3.3 (S), R9.1
- new net: JP1.2 (B), Q3.3 (S), R9.1
Other:
- moved on the sheet: C12, C13
Changed lines of the file:
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@@
 	)
 	(junction
-		(at 152.4 69.85)
+		(at 139.7 59.69)
 		(diameter 0)
 		(color 0 0 0 0)
 	)
 	(junction
-		(at 152.4 49.53)
+		(at 204.47 49.53)
 		(diameter 0)
 		(color 0 0 0 0)
 	)
 	(junction
-		(at 139.7 59.69)
+		(at 218.44 69.85)
 		(diameter 0)
 		(color 0 0 0 0)
 	)
 	(junction
-		(at 204.47 49.53)
+		(at 139.7 69.85)
 		(diameter 0)
 		(color 0 0 0 0)
 	)
 	(junction
-		(at 218.44 69.85)
+		(at 134.62 49.53)
 		(diameter 0)
 		(color 0 0 0 0)
 	)
 	(junction
-		(at 139.7 69.85)
+		(at 162.56 49.53)
 		(diameter 0)
 		(color 0 0 0 0)
 	)
 	(junction
-		(at 134.62 49.53)
+		(at 218.44 49.53)
 		(diameter 0)
 		(color 0 0 0 0)
 	)
 	(junction
-		(at 218.44 49.53)
+		(at 179.07 49.53)
 		(diameter 0)
 		(color 0 0 0 0)
@@
 	)
 	(junction
-		(at 71.12 124.46)
+		(at 149.86 49.53)
 		(diameter 0)
 		(color 0 0 0 0)
 	)
 	(junction
-		(at 82.55 69.85)
+		(at 71.12 124.46)
 		(diameter 0)
 		(color 0 0 0 0)
 	)
 	(junction
-		(at 165.1 49.53)
+		(at 82.55 69.85)
 		(diameter 0)
 		(color 0 0 0 0)
 	)
 	(junction
-		(at 66.04 69.85)
+		(at 149.86 69.85)
 		(diameter 0)
 		(color 0 0 0 0)
 	)
 	(junction
-		(at 69.85 49.53)
+		(at 66.04 69.85)
 		(diameter 0)
 		(color 0 0 0 0)
 	)
 	(junction
-		(at 179.07 49.53)
+		(at 69.85 49.53)
 		(diameter 0)
 		(color 0 0 0 0)
@@
 	(wire
 		(pts
-			(xy 95.25 52.07) (xy 102.87 52.07)
+			(xy 175.26 49.53) (xy 179.07 49.53)
 		)
 		(stroke
@@
 	(wire
 		(pts
-			(xy 179.07 49.53) (xy 165.1 49.53)
+			(xy 95.25 52.07) (xy 102.87 52.07)
 		)
 		(stroke
@@
 	(wire
 		(pts
-			(xy 165.1 69.85) (xy 152.4 69.85)
+			(xy 139.7 59.69) (xy 139.7 60.96)
 		)
 		(stroke
@@
 	(wire
 		(pts
-			(xy 139.7 59.69) (xy 139.7 60.96)
+			(xy 139.7 59.69) (xy 139.7 58.42)
 		)
 		(stroke
@@
 	(wire
 		(pts
-			(xy 139.7 59.69) (xy 139.7 58.42)
+			(xy 149.86 49.53) (xy 139.7 49.53)
+		)
+		(stroke
+			(width 0)
+			(type default)
+		)
+	)
+	(wire
+		(pts
+			(xy 149.86 69.85) (xy 162.56 69.85)
 		)
 		(stroke
@@
 	(wire
 		(pts
+			(xy 162.56 49.53) (xy 165.1 49.53)
+		)
+		(stroke
+			(width 0)
+			(type default)
+		)
+	)
+	(wire
+		(pts
 			(xy 134.62 49.53) (xy 134.62 52.07)
 		)
@@
 	(wire
 		(pts
-			(xy 139.7 69.85) (xy 152.4 69.85)
+			(xy 139.7 69.85) (xy 149.86 69.85)
 		)
 		(stroke
@@
 	(wire
 		(pts
-			(xy 165.1 36.83) (xy 165.1 49.53)
+			(xy 162.56 36.83) (xy 162.56 49.53)
 		)
 		(stroke
@@
 	(wire
 		(pts
-			(xy 165.1 36.83) (xy 168.91 36.83)
+			(xy 162.56 36.83) (xy 168.91 36.83)
 		)
 		(stroke
@@
 	(wire
 		(pts
-			(xy 165.1 49.53) (xy 165.1 55.88)
+			(xy 162.56 49.53) (xy 162.56 55.88)
 		)
 		(stroke
@@
 	(wire
 		(pts
-			(xy 152.4 49.53) (xy 139.7 49.53)
+			(xy 149.86 49.53) (xy 162.56 49.53)
 		)
 		(stroke
@@
 	(wire
 		(pts
-			(xy 165.1 49.53) (xy 152.4 49.53)
-		)
-		(stroke
-			(width 0)
-			(type default)
-		)
-	)
-	(wire
-		(pts
 			(xy 204.47 63.5) (xy 204.47 69.85)
 		)
@@
 	(wire
 		(pts
-			(xy 165.1 63.5) (xy 165.1 69.85)
+			(xy 162.56 63.5) (xy 162.56 69.85)
 		)
 		(stroke
@@
 	(wire
 		(pts
-			(xy 152.4 63.5) (xy 152.4 69.85)
+			(xy 149.86 63.5) (xy 149.86 69.85)
 		)
 		(stroke
@@
 	(wire
 		(pts
-			(xy 152.4 55.88) (xy 152.4 49.53)
+			(xy 149.86 55.88) (xy 149.86 49.53)
 		)
 		(stroke
@@
 	(symbol
 		(lib_id "Device:C_Polarized")
-		(at 152.4 59.69 0)
+		(at 149.86 59.69 0)
 		(unit 1)
 		(exclude_from_sim no)
@@
 		(fields_autoplaced yes)
 		(property "Reference" "C12"
-			(at 156.21 57.5309 0)
+			(at 153.67 57.5309 0)
 			(effects
 				(font
@@
 		)
 		(property "Value" "100µF"
-			(at 156.21 60.0709 0)
+			(at 153.67 60.0709 0)
 			(effects
 				(font
@@
 		)
 		(property "Footprint" "CollecteurDonne:C_Radial_D10.0mm_H16.0mm_P5.00mm"
-			(at 153.3652 63.5 0)
+			(at 150.8252 63.5 0)
 			(effects
 				(font
@@
 		)
 		(property "Datasheet" "~"
-			(at 152.4 59.69 0)
+			(at 149.86 59.69 0)
 			(effects
 				(font
@@
 		)
 		(property "Description" "Polarized capacitor"
-			(at 152.4 59.69 0)
+			(at 149.86 59.69 0)
 			(effects
 				(font
@@
 		)
 		(property "Fabricant" "Vishay"
-			(at 152.4 59.69 0)
+			(at 149.86 59.69 0)
 			(effects
 				(font
@@
 		)
 		(property "Fournisseur" "RS"
-			(at 152.4 59.69 0)
+			(at 149.86 59.69 0)
 			(effects
 				(font
@@
 		)
 		(property "Ref Fabricant" "MAL215373101E3"
-			(at 152.4 59.69 0)
+			(at 149.86 59.69 0)
 			(effects
 				(font
@@
 		)
 		(property "Ref Fournisseur" "280-6780P"
-			(at 152.4 59.69 0)
+			(at 149.86 59.69 0)
 			(effects
 				(font
@@
 		)
 		(property "Sim.Type" ""
-			(at 152.4 59.69 0)
+			(at 149.86 59.69 0)
 			(effects
 				(font
@@
 	)
 	(symbol
+		(lib_id "Jumper:Jumper_2_Bridged")
+		(at 170.18 49.53 0)
+		(unit 1)
+		(exclude_from_sim no)
+		(in_bom yes)
+		(on_board yes)
+		(dnp no)
+		(property "Reference" "JP1"
+			(at 172.72 42.164 0)
+			(effects
+				(font
+					(size 1.27 1.27)
+				)
+			)
+		)
+		(property "Value" "Jumper_2_Bridged"
+			(at 172.72 44.704 0)
+			(effects
+				(font
+					(size 1.27 1.27)
+				)
+			)
+		)
+		(property "Footprint" "Connector_PinHeader_2.54mm:PinHeader_1x02_P2.54mm_Vertical"
+			(at 170.18 49.53 0)
+			(effects
+				(font
+					(size 1.27 1.27)
+				)
+				(hide yes)
+			)
+		)
+		(property "Datasheet" "~"
+			(at 170.18 49.53 0)
+			(effects
+				(font
+					(size 1.27 1.27)
+				)
+				(hide yes)
+			)
+		)
+		(property "Description" "Jumper, 2-pole, closed/bridged"
+			(at 170.18 49.53 0)
+			(effects
+				(font
+					(size 1.27 1.27)
+				)
+				(hide yes)
+			)
+		)
+		(pin "1"
+		)
+		(pin "2"
+		)
+		(instances
+			(project ""
+				(path "/77f264da-4c84-4b0c-9d20-4392731765e6/8078826c-4446-4e50-a209-45fcf7cbe7e4"
+					(reference "JP1")
+					(unit 1)
+				)
+			)
+		)
+	)
+	(symbol
 		(lib_id "Connector:Screw_Terminal_01x02")
 		(at 252.73 25.4 0)
@@
 	(symbol
 		(lib_id "Device:C")
-		(at 165.1 59.69 0)
+		(at 162.56 59.69 0)
 		(unit 1)
 		(exclude_from_sim no)
@@
 		(dnp no)
 		(property "Reference" "C13"
-			(at 168.91 58.4199 0)
+			(at 166.37 58.4199 0)
 			(effects
 				(font
@@
 		)
 		(property "Value" "100nF"
-			(at 168.91 60.96 0)
+			(at 166.37 60.96 0)
 			(effects
 				(font
@@
 		)
 		(property "Footprint" "CollecteurDonne:C_Disc_D5.0mm_W2.5mm_P5.00mm"
-			(at 166.0652 63.5 0)
+			(at 163.5252 63.5 0)
 			(effects
 				(font
@@
 		)
 		(property "Datasheet" "~"
-			(at 165.1 59.69 0)
+			(at 162.56 59.69 0)
 			(effects
 				(font
@@
 		)
 		(property "Description" "Unpolarized capacitor"
-			(at 165.1 59.69 0)
+			(at 162.56 59.69 0)
 			(effects
 				(font
@@
 		)
 		(property "Fabricant" "KEMET"
-			(at 165.1 59.69 0)
+			(at 162.56 59.69 0)
 			(effects
 				(font
@@
 		)
 		(property "Fournisseur" "RS"
-			(at 165.1 59.69 0)
+			(at 162.56 59.69 0)
 			(effects
 				(font
@@
 		)
 		(property "Ref Fabricant" "C0805C104K4RACTU"
-			(at 165.1 59.69 0)
+			(at 162.56 59.69 0)
 			(effects
 				(font
@@
 		)
 		(property "Ref Fournisseur" "648-0957"
-			(at 165.1 59.69 0)
+			(at 162.56 59.69 0)
 			(effects
 				(font
@@
 		)
 		(property "Sim.Type" ""
-			(at 165.1 59.69 0)
+			(at 162.56 59.69 0)
 			(effects
 				(font

Commit message: Update_6_02_2026
Parts:
- C12: value 100µF -> 470µF
Changed lines of the file:
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@@
 			)
 		)
-		(property "Value" "100µF"
+		(property "Value" "470µF"
 			(at 153.67 60.0709 0)
 			(effects

Commit message: Update
Other:
- note added: "MAUVAISE EMPREINTE INDUCTOR"
Changed lines of the file:
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@@
+	)
+	(rectangle
+		(start 106.68 29.21)
+		(end 144.78 54.61)
+		(stroke
+			(width 0.635)
+			(type solid)
+			(color 255 0 2 1)
+		)
+		(fill
+			(type none)
+		)
 	)
 	(rectangle
@@
 			)
 		)
+	)
+	(text "MAUVAISE EMPREINTE INDUCTOR\n"
+		(exclude_from_sim no)
+		(at 126.746 34.798 0)
+		(effects
+			(font
+				(size 1.27 1.27)
+				(color 255 50 6 1)
+			)
+		)
