File: Architecture/Main-REVA2/Power.kicad_sch (KiCad schematic)
At the start: 27 parts, among them J10 IN, J14 OUT_5V_ALI, J16 OUT_5V_PWR, J17 Barrel_Jack_Switch_Pin3Ring, Q2 PN2222A, Q3 IRF9540N, U3 MCP16311x-xMS

Commit message: Update_09_04_2026_PC
Other:
- note removed: "https://www.microchip.com/en-us/parametric-search/418?filters=JTdCJTIyYWN0aXZlU2xpZGVyRmlsdGVycyUyMiUzQSU1QiU1QiUyMlZJTiUyME1pbiUyMFYlMjAodm9sdCklMjIlMkMlNUI0LjIlMkMyLjIlNUQlNUQlNUQlMkMlMjJjYXRlZ29yeWRyb3Bkb3duJTIyJTNBJTVCJTIyUG93ZXIlMjBNYW5hZ2VtZW50JTIyJTJDJTIyREMtREMlMjBCb29zdCUyMChTdGVwLVVwKSUyMFN3aXRjaGluZyUyMENvbnZlcnRlcnMlMjIlMkMlMjJCdWNrJTIwU3dpdGNoaW5nJTIwQ29udmVydGVycyUyMCVFMiU4MCU5MyUyM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"
Changed lines of the file:
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@@
-		)
-	)
-	(text "https://www.microchip.com/en-us/parametric-search/418?filters=JTdCJTIyYWN0aXZlU2xpZGVyRmlsdGVycyUyMiUzQSU1QiU1QiUyMlZJTiUyME1pbiUyMFYlMjAodm9sdCklMjIlMkMlNUI0LjIlMkMyLjIlNUQlNUQlNUQlMkMlMjJjYXRlZ29yeWRyb3Bkb3duJTIyJTNBJTVCJTIyUG93ZXIlMjBNYW5hZ2VtZW50JTIyJTJDJTIyREMtREMlMjBCb29zdCUyMChTdGVwLVVwKSUyMFN3aXRjaGluZyUyMENvbnZlcnRlcnMlMjIlMkMlMjJCdWNrJTIwU3dpdGNoaW5nJTIwQ29udmVydGVycyUyMCVFMiU4MCU5MyUyMFN0ZXAlMjBEb3duJTIwKDEwViUyMHRvJTIwMzZWKSUyMiU1RCU3RA=="
-		(exclude_from_sim no)
-		(at 155.702 -12.192 0)
-		(effects
-			(font
-				(size 1.27 1.27)
-			)
 		)
 	)
