File: Architecture/Main-REVA2/Sensors.kicad_sch (KiCad schematic)
At the start: 9 parts, among them J3 Conn_01x03, J4 Conn_01x04, J6 Conn_01x04

Commit message: Update_Schematic
Parts:
- removed R4: 10k, symbol Device:R_US
- added C6: 100nF, symbol Device:C
- added J7, J8: Conn_01x06, symbol Connector_Generic:Conn_01x06
- added Q1: NMOS, symbol Simulation_SPICE:NMOS
- R3: value 10k -> 1k
Connections:
- net +3.3V_BATTERY is gone; now on net +VCC: J3.1 (Pin_1)
- net GND: now also C6.2, J7.1 (Pin_1), J8.2 (Pin_2); no longer C2.2, J6.4 (Pin_4)
- net I2C_SCL: now also J8.3 (Pin_3)
- net I2C_SDA: now also J8.4 (Pin_4)
- net RX0: now also J7.5 (Pin_5)
- net TX0: now also J7.4 (Pin_4)
- net +3.3V renamed +VCC
- net +VCC: now also C6.1, J7.3 (Pin_3), J8.1 (Pin_1)
- net Voltage_Batt renamed ENA_GPS
- net Voltage_Batt_value: no longer names the net of R3.2
- net Voltage_Batt_value: now also Q1.2 (G)
- new net: J6.4 (Pin_4), J7.6 (Pin_6), Q1.1 (D)
- new net: C2.2, Q1.3 (S)
- no-connect marks 1 -> 4
Other:
- note added: "BME680"
- note added: "BME680 - Temp;Hum;Press;Qual"
- note added: "BN220"
- note added: "PA1010D"
- note added: "WAKE"
- note removed: "Battery Voltage"
- company: (none) -> Polytech Nantes - ETN4
- title: (none) -> Collecteur de données Animalières
- moved on the sheet: C2, C3, J3, J4, J6, R5, R6

Commit message: Update
Parts:
- removed Q1: NMOS, symbol Simulation_SPICE:NMOS
- added C16, C17, C18, C19: 100nF, Capacitor_THT:C_Disc_D4.3mm_W1.9mm_P5.00mm, symbol Device:C
- added J12, J13, J15: Conn_01x04, symbol Connector_Generic:Conn_01x04
- added Q1: BS170, Package_TO_SOT_THT:TO-92_Inline, symbol Transistor_FET:BS170
- C2, C3, C6: footprint (none) -> Capacitor_THT:C_Disc_D4.3mm_W1.9mm_P5.00mm; Fabricant (none) -> KEMET; Fournisseur (none) -> RS; Ref Fabricant (none) -> C0805C104K4RACTU; Ref Fournisseur (none) -> 648-0957
- J3: footprint (none) -> Connector_PinHeader_2.54mm:PinHeader_1x03_P2.54mm_Vertical
- J6: footprint (none) -> Connector_PinHeader_2.54mm:PinHeader_1x04_P2.54mm_Vertical
- J7, J8: footprint (none) -> Connector_PinHeader_2.54mm:PinHeader_1x06_P2.54mm_Vertical
- R5: Fournisseur (none) -> Gotronic; Ref Fournisseur (none) -> 03131
Connections:
- net +VCC: now also C16.1, C17.1, C18.1, C19.1, J12.2 (Pin_2), J13.2 (Pin_2), J15.2 (Pin_2)
- net GND: now also J6.4 (Pin_4), C16.2, C17.2, C18.2, C19.2, J12.1 (Pin_1), J13.1 (Pin_1), J15.1 (Pin_1), Q1.1 (D)
- net I2C_SCL: now also J12.4 (Pin_4), J13.4 (Pin_4), J15.4 (Pin_4)
- net I2C_SDA: now also J12.3 (Pin_3), J13.3 (Pin_3), J15.3 (Pin_3)
- net at J7.6 (Pin_6): no longer J6.4 (Pin_4)
- net at R3.2: now also Q1.2 (G)
- net at C2.2: now also Q1.3 (S)
- no-connect marks 4 -> 5
Other:
- note added: "Brightness Sensor ( I/O D__ )"
- note added: "I2C_Sensor_Gravity"
- note added: "I2C_Sensor_Groove"
- note added: "I2C_Sensor_Header"
- note added: "PPS"
- note removed: "Brightness Sensor ( I/O D36 )"
- moved on the sheet: C6, J3, J8

Commit message: Update_Sche
Parts:
- C16, C17, C18, C19, C2, C3, C6: footprint Capacitor_THT:C_Disc_D4.3mm_W1.9mm_P5.00mm -> CollecteurDonne:Capa disc radial 5.08mm
- R3, R6: footprint (none) -> CollecteurDonne:Résistance L10mm
- R5: footprint OptoDevice:R_LDR_10x8.5mm_P7.6mm_Vertical -> CollecteurDonne:Résistance L10mm
Changed lines of the file:
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@@
 			)
 		)
-		(property "Footprint" "OptoDevice:R_LDR_10x8.5mm_P7.6mm_Vertical"
+		(property "Footprint" "CollecteurDonne:Résistance L10mm"
 			(at 113.665 49.53 90)
 			(effects
@@
 			)
 		)
-		(property "Footprint" "Capacitor_THT:C_Disc_D4.3mm_W1.9mm_P5.00mm"
+		(property "Footprint" "CollecteurDonne:Capa disc radial 5.08mm"
 			(at 210.5152 100.33 0)
 			(effects
@@
 			)
 		)
-		(property "Footprint" "Capacitor_THT:C_Disc_D4.3mm_W1.9mm_P5.00mm"
+		(property "Footprint" "CollecteurDonne:Capa disc radial 5.08mm"
 			(at 136.8552 143.51 0)
 			(effects
@@
 			)
 		)
-		(property "Footprint" "Capacitor_THT:C_Disc_D4.3mm_W1.9mm_P5.00mm"
+		(property "Footprint" "CollecteurDonne:Capa disc radial 5.08mm"
 			(at 131.7752 101.6 0)
 			(effects
@@
 			)
 		)
-		(property "Footprint" "Capacitor_THT:C_Disc_D4.3mm_W1.9mm_P5.00mm"
+		(property "Footprint" "CollecteurDonne:Capa disc radial 5.08mm"
 			(at 65.7352 99.06 0)
 			(effects
@@
 			)
 		)
-		(property "Footprint" "Capacitor_THT:C_Disc_D4.3mm_W1.9mm_P5.00mm"
+		(property "Footprint" "CollecteurDonne:Capa disc radial 5.08mm"
 			(at 55.5752 143.51 0)
 			(effects
@@
 			)
 		)
-		(property "Footprint" ""
+		(property "Footprint" "CollecteurDonne:Résistance L10mm"
 			(at 169.164 63.754 90)
 			(effects
@@
 			)
 		)
-		(property "Footprint" ""
+		(property "Footprint" "CollecteurDonne:Résistance L10mm"
 			(at 110.236 59.944 90)
 			(effects
@@
 			)
 		)
-		(property "Footprint" "Capacitor_THT:C_Disc_D4.3mm_W1.9mm_P5.00mm"
+		(property "Footprint" "CollecteurDonne:Capa disc radial 5.08mm"
 			(at 218.1352 143.51 0)
 			(effects
@@
 			)
 		)
-		(property "Footprint" "Capacitor_THT:C_Disc_D4.3mm_W1.9mm_P5.00mm"
+		(property "Footprint" "CollecteurDonne:Capa disc radial 5.08mm"
 			(at 174.9552 55.88 0)
 			(effects

Commit message: Update_Schematic_PCB
Parts:
- removed J12, J15: Conn_01x04, symbol Connector_Generic:Conn_01x04
- removed R5: LDR03, CollecteurDonne:Résistance L10mm, symbol Sensor_Optical:LDR03
- removed R6: 10k, CollecteurDonne:Résistance L10mm, symbol Device:R_US
- added J11, J12: 110990030, 110990030:SEEED_110990030, symbol Grove:110990030
- C16, C17, C18, C19, C2, C6: footprint CollecteurDonne:Capa disc radial 5.08mm -> CollecteurDonne:C_Disc_D5.0mm_W2.5mm_P5.00mm
- C3: footprint CollecteurDonne:Capa disc radial 5.08mm -> CollecteurDonne:C_Disc_D5.0mm_W2.5mm_P5.00mm; now not fitted
- J13: footprint (none) -> Connector_PinHeader_2.54mm:PinHeader_1x04_P2.54mm_Vertical
- J4: now not fitted
- R3: footprint CollecteurDonne:Résistance L10mm -> CollecteurDonne:R_Axial_DIN0207_L6.3mm_D2.5mm_P10.16mm_Horizontal
Connections:
- net +VCC: now also J11.2, J12.2
- net GND: now also J11.1, J12.1
- net I2C_SCL: now also J11.4, J12.4
- net I2C_SDA: now also J11.3, J12.3
Other:
- note removed: "Brightness Sensor ( I/O D__ )"
- note removed: "I2C_Sensor_Gravity"
- moved on the sheet: C16, C17, C18, C19, C2, C6, J13, J3, J6, J7, J8, Q1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

Commit message: Update_28_01_2025
Parts:
- removed C18: 100nF, CollecteurDonne:C_Disc_D5.0mm_W2.5mm_P5.00mm, symbol Device:C
- removed J13: Conn_01x04, Connector_PinHeader_2.54mm:PinHeader_1x04_P2.54mm_Vertical, symbol Connector_Generic:Conn_01x04
Other:
- note removed: "I2C_Sensor_Header"
- moved on the sheet: C16, C17, J11, J12

Commit message: Update_PCB
Parts:
- removed Q1: BS170, Package_TO_SOT_THT:TO-92_Inline, symbol Transistor_FET:BS170
- added Q1: IRF540N, Package_TO_SOT_THT:TO-220-3_Vertical, symbol Transistor_FET:IRF540N
- J11, J12: footprint 110990030:SEEED_110990030 -> CollecteurDonne:Grove
- J4: footprint (none) -> Connector_PinHeader_2.54mm:PinHeader_1x04_P2.54mm_Vertical
Connections:
- net GND: now also Q1.2 (D)
- net at R3.2: now also Q1.1 (G)
- net at C2.2: now also Q1.3 (S)
Changed lines of the file:
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@@
 			)
 		)
-		(property "Footprint" "110990030:SEEED_110990030"
+		(property "Footprint" "CollecteurDonne:Grove"
 			(at 201.93 133.35 0)
 			(effects
@@
 			)
 		)
-		(property "Footprint" "110990030:SEEED_110990030"
+		(property "Footprint" "CollecteurDonne:Grove"
 			(at 119.38 133.35 0)
 			(effects
@@
 			)
 		)
-		(property "Footprint" ""
+		(property "Footprint" "Connector_PinHeader_2.54mm:PinHeader_1x04_P2.54mm_Vertical"
 			(at 166.37 88.9 0)
 			(effects
@@
 	)
 	(symbol
+		(lib_id "Transistor_FET:IRF540N")
+		(at 142.24 59.69 0)
+		(unit 1)
+		(exclude_from_sim no)
+		(in_bom yes)
+		(on_board yes)
+		(dnp no)
+		(fields_autoplaced yes)
+		(property "Reference" "Q1"
+			(at 148.59 58.4199 0)
+			(effects
+				(font
+					(size 1.27 1.27)
+				)
+				(justify left)
+			)
+		)
+		(property "Value" "IRF540N"
+			(at 148.59 60.9599 0)
+			(effects
+				(font
+					(size 1.27 1.27)
+				)
+				(justify left)
+			)
+		)
+		(property "Footprint" "Package_TO_SOT_THT:TO-220-3_Vertical"
+			(at 147.32 61.595 0)
+			(effects
+				(font
+					(size 1.27 1.27)
+					(italic yes)
+				)
+				(justify left)
+				(hide yes)
+			)
+		)
+		(property "Datasheet" "http://www.irf.com/product-info/datasheets/data/irf540n.pdf"
+			(at 147.32 63.5 0)
+			(effects
+				(font
+					(size 1.27 1.27)
+				)
+				(justify left)
+				(hide yes)
+			)
+		)
+		(property "Description" "33A Id, 100V Vds, HEXFET N-Channel MOSFET, TO-220"
+			(at 142.24 59.69 0)
+			(effects
+				(font
+					(size 1.27 1.27)
+				)
+				(hide yes)
+			)
+		)
+		(pin "2"
+		)
+		(pin "1"
+		)
+		(pin "3"
+		)
+		(instances
+			(project "Main"
+				(path "/77f264da-4c84-4b0c-9d20-4392731765e6/1ddae4dd-6d7b-4ef8-9a8d-fbd44b538466"
+					(reference "Q1")
+					(unit 1)
+				)
+			)
+		)
+	)
+	(symbol
 		(lib_id "Device:C")
 		(at 176.53 134.62 0)
@@
 					(unit 1)
 				)
-			)
-		)
-	)
-	(symbol
-		(lib_id "Transistor_FET:BS170")
-		(at 142.24 59.69 0)
-		(unit 1)
-		(exclude_from_sim no)
-		(in_bom yes)
-		(on_board yes)
-		(dnp no)
-		(fields_autoplaced yes)
-		(property "Reference" "Q1"
-			(at 148.59 58.4199 0)
-			(effects
-				(font
-					(size 1.27 1.27)
-				)
-				(justify left)
-			)
-		)
-		(property "Value" "BS170"
-			(at 148.59 60.9599 0)
-			(effects
-				(font
-					(size 1.27 1.27)
-				)
-				(justify left)
-			)
-		)
-		(property "Footprint" "Package_TO_SOT_THT:TO-92_Inline"
-			(at 147.32 61.595 0)
-			(effects
-				(font
-					(size 1.27 1.27)
-					(italic yes)
-				)
-				(justify left)
-				(hide yes)
-			)
-		)
-		(property "Datasheet" "https://www.onsemi.com/pub/Collateral/BS170-D.PDF"
-			(at 147.32 63.5 0)
-			(effects
-				(font
-					(size 1.27 1.27)
-				)
-				(justify left)
-				(hide yes)
-			)
-		)
-		(property "Description" "0.5A Id, 60V Vds, N-Channel MOSFET, TO-92"
-			(at 142.24 59.69 0)
-			(effects
-				(font
-					(size 1.27 1.27)
-				)
-				(hide yes)
-			)
-		)
-		(property "Fabricant" "BS170"
-			(at 142.24 59.69 0)
-			(effects
-				(font
-					(size 1.27 1.27)
-				)
-				(hide yes)
-			)
-		)
-		(property "Fournisseur" "RS"
-			(at 142.24 59.69 0)
-			(effects
-				(font
-					(size 1.27 1.27)
-				)
-				(hide yes)
-			)
-		)
-		(property "Ref Fabricant" "ONSEMI"
-			(at 142.24 59.69 0)
-			(effects
-				(font
-					(size 1.27 1.27)
-				)
-				(hide yes)
-			)
-		)
-		(property "Ref Fournisseur" "124-1745"
-			(at 142.24 59.69 0)
-			(effects
-				(font
-					(size 1.27 1.27)
-				)
-				(hide yes)
-			)
-		)
-		(property "Sim.Type" ""
-			(at 142.24 59.69 0)
-			(effects
-				(font
-					(size 1.27 1.27)
-				)
-				(hide yes)
-			)
-		)
-		(pin "2"
-		)
-		(pin "3"
-		)
-		(pin "1"
-		)
-		(instances
-			(project "Main"
-				(path "/77f264da-4c84-4b0c-9d20-4392731765e6/1ddae4dd-6d7b-4ef8-9a8d-fbd44b538466"
-					(reference "Q1")
-					(unit 1)
-				)

Commit message: Update_6_02_2026
Parts:
- added R6: 10k, CollecteurDonne:R_Axial_DIN0207_L6.3mm_D2.5mm_P10.16mm_Horizontal, symbol Device:R_US
Connections:
- net GND: now also R6.2
- net PIR_MOUV: now also R6.1
Changed lines of the file:
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@@
 	)
 	(junction
+		(at 49.53 90.17)
+		(diameter 0)
+		(color 0 0 0 0)
+	)
+	(junction
 		(at 144.78 52.07)
 		(diameter 0)
@@
 	(wire
 		(pts
-			(xy 80.01 90.17) (xy 86.36 90.17)
+			(xy 46.99 90.17) (xy 49.53 90.17)
+		)
+		(stroke
+			(width 0)
+			(type default)
+		)
+	)
+	(wire
+		(pts
+			(xy 49.53 100.33) (xy 49.53 101.6)
 		)
 		(stroke
@@
 	(wire
 		(pts
+			(xy 49.53 90.17) (xy 86.36 90.17)
+		)
+		(stroke
+			(width 0)
+			(type default)
+		)
+	)
+	(wire
+		(pts
 			(xy 107.95 138.43) (xy 109.22 138.43)
 		)
@@
 	(wire
 		(pts
+			(xy 49.53 90.17) (xy 49.53 92.71)
+		)
+		(stroke
+			(width 0)
+			(type default)
+		)
+	)
+	(wire
+		(pts
 			(xy 224.79 93.98) (xy 227.33 93.98)
 		)
@@
 	(wire
 		(pts
+			(xy 49.53 101.6) (xy 66.04 101.6)
+		)
+		(stroke
+			(width 0)
+			(type default)
+		)
+	)
+	(wire
+		(pts
 			(xy 172.72 50.8) (xy 175.26 50.8)
 		)
@@
 	(wire
 		(pts
+			(xy 66.04 101.6) (xy 66.04 93.98)
+		)
+		(stroke
+			(width 0)
+			(type default)
+		)
+	)
+	(wire
+		(pts
 			(xy 142.24 48.26) (xy 147.32 48.26)
 		)
@@
 	(hierarchical_label "PIR_MOUV"
 		(shape input)
-		(at 80.01 90.17 180)
+		(at 46.99 90.17 180)
 		(effects
 			(font
@@
 					(unit 1)
 				)
+			)
+		)
+	)
+	(symbol
+		(lib_id "Device:R_US")
+		(at 49.53 96.52 0)
+		(unit 1)
+		(exclude_from_sim no)
+		(in_bom yes)
+		(on_board yes)
+		(dnp no)
+		(fields_autoplaced yes)
+		(property "Reference" "R6"
+			(at 52.07 95.2499 0)
+			(effects
+				(font
+					(size 1.27 1.27)
+				)
+				(justify left)
+			)
+		)
+		(property "Value" "10k"
+			(at 52.07 97.7899 0)
+			(effects
+				(font
+					(size 1.27 1.27)
+				)
+				(justify left)
+			)
+		)
+		(property "Footprint" "CollecteurDonne:R_Axial_DIN0207_L6.3mm_D2.5mm_P10.16mm_Horizontal"
+			(at 50.546 96.774 90)
+			(effects
+				(font
+					(size 1.27 1.27)
+				)
+				(hide yes)
+			)
+		)
+		(property "Datasheet" "~"
+			(at 49.53 96.52 0)
+			(effects
+				(font
+					(size 1.27 1.27)
+				)
+				(hide yes)
+			)
+		)
+		(property "Description" "Resistor, US symbol"
+			(at 49.53 96.52 0)
+			(effects
+				(font
+					(size 1.27 1.27)
+				)
+				(hide yes)
+			)
+		)
+		(pin "2"
+		)
+		(pin "1"
+		)
+		(instances
+			(project ""
+				(path "/77f264da-4c84-4b0c-9d20-4392731765e6/1ddae4dd-6d7b-4ef8-9a8d-fbd44b538466"
+					(reference "R6")
+					(unit 1)
+				)

Commit message: Update
Parts:
- added D4: LED, LED_THT:LED_D5.0mm, symbol Device:LED
- added Q5: PN2222A, Package_TO_SOT_THT:TO-92_Inline, symbol Transistor_BJT:PN2222A
- added R12: 10k, CollecteurDonne:R_Axial_DIN0207_L6.3mm_D2.5mm_P10.16mm_Horizontal, symbol Device:R_US
- added R13: 1k, CollecteurDonne:R_Axial_DIN0207_L6.3mm_D2.5mm_P10.16mm_Horizontal, symbol Device:R_US
Connections:
- net +VCC: now also R12.1
- net GND: now also Q5.1 (E)
- new net: Q5.2 (B), R13.2
- new net: D4.1 (K), Q5.3 (C)
- new net: D4.2 (A), R12.2
- new net DEBUG: R13.1
Other:
- note added: "DEBUG MODE"
- note added: "ERREUR NON VCC => V Battery"
- moved on the sheet: C2, J6, J7, Q1, R3
